File: Projects/KiCad/THRControlModuleBoard/THRControlModuleBoard.kicad_sch (KiCad schematic)
At the start: 26 parts, among them J1 Conn_01x02_Socket, J2 Conn_01x02_Socket, J3 Screw_Terminal_01x02, Q1 Q_PMOS_GDS, Q2 Q_PMOS_GDS, Q3 Q_PMOS_GDS, U1 LTC4416EMS#PBF, U2 MAX31856MUD+T

Commit message: THRControlModuleBoard
Parts:
- C3, C4, C5, C6, C7: footprint (none) -> Capacitor_SMD:C_0805_2012Metric_Pad1.18x1.45mm_HandSolder
- D1, D2, D3: footprint (none) -> Diode_SMD:D_0805_2012Metric_Pad1.15x1.40mm_HandSolder
- R4, R5, R6, R7, R8: footprint (none) -> Resistor_SMD:R_0805_2012Metric_Pad1.20x1.40mm_HandSolder
- U2: footprint Package_SO:SOP65P640X110-14N -> Package_SO:TSSOP-14_4.4x5mm_P0.65mm
Connections:
- net GND: no longer U1.4 (*E2)
- net QMOS/3-3: now reaches Q1.3 (S), Q2.3 (S)
- no-connect marks 1 -> 2

Commit message: THRControlModuleBoardに熱電対アンプモジュールを追加しました。
Parts:
- J3: footprint (none) -> TerminalBlock:TerminalBlock_Altech_AK300-2_P5.00mm
Connections:
- net at R4.2, U2.3 (T-): now also C5.2, C7.1
- net THERM+: no longer names the net of J3.2 (Pin_2), R5.1
Changed lines of the file:
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@@
   (junction (at 121.92 49.53) (diameter 0) (color 0 0 0 0)
+  )
+  (junction (at 121.92 62.23) (diameter 0) (color 0 0 0 0)
   )
   (junction (at 224.79 137.16) (diameter 0) (color 0 0 0 0)
@@
     (stroke (width 0) (type default))
   )
+  (wire (pts (xy 121.92 62.23) (xy 121.92 64.77))
+    (stroke (width 0) (type default))
+  )
   (wire (pts (xy 104.14 54.61) (xy 106.68 54.61))
     (stroke (width 0) (type default))
@@
     (stroke (width 0) (type default))
   )
-  (wire (pts (xy 121.92 59.69) (xy 121.92 64.77))
+  (wire (pts (xy 121.92 59.69) (xy 121.92 62.23))
     (stroke (width 0) (type default))
   )
@@
     (stroke (width 0) (type default))
   )
+  (wire (pts (xy 121.92 62.23) (xy 118.11 62.23))
+    (stroke (width 0) (type default))
+  )
   (wire (pts (xy 39.37 125.73) (xy 39.37 127))
     (stroke (width 0) (type default))
@@
     (stroke (width 0) (type default))
   )
-  (wire (pts (xy 130.81 62.23) (xy 118.11 62.23))
+  (wire (pts (xy 130.81 62.23) (xy 121.92 62.23))
     (stroke (width 0) (type default))
   )
@@
   )
   (label "QMOS{slash}3-3" (at 205.74 113.03 0) (fields_autoplaced)
-    (effects (font (size 1.27 1.27)) (justify left bottom))
-  )
-  (label "THERM-" (at 106.68 62.23 180) (fields_autoplaced)
-    (effects (font (size 1.27 1.27)) (justify right bottom))
-  )
-  (label "THERM+" (at 106.68 54.61 0) (fields_autoplaced)
     (effects (font (size 1.27 1.27)) (justify left bottom))
   )
@@
       (effects (font (size 1.27 1.27)))
     )
-    (property "Footprint" "" (at 99.06 57.15 0)
-      (effects (font (size 1.27 1.27)) hide)
-    )
+    (property "Footprint" "TerminalBlock:TerminalBlock_Altech_AK300-2_P5.00mm" (at 99.06 57.15 0)
+      (effects (font (size 1.27 1.27)) hide)
+    )

Commit message: THRControlModuleBoardの更新
Changed lines of the file:
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@@
   (junction (at 209.55 64.77) (diameter 0) (color 0 0 0 0)
-  )
-  (junction (at 187.96 49.53) (diameter 0) (color 0 0 0 0)
   )
   (junction (at 189.23 120.65) (diameter 0) (color 0 0 0 0)
@@
         (path "/79fd2516-dad6-414c-bb46-91ee9bfb5006"
           (reference "R5") (unit 1)
-        )
-      )
-    )
-  )
-  (symbol (lib_id "power:PWR_FLAG") (at 187.96 49.53 270) (unit 1)
-    (in_bom yes) (on_board yes) (dnp no)
-    (property "Reference" "#FLG02" (at 189.865 49.53 0)
-      (effects (font (size 1.27 1.27)) hide)
-    )
-    (property "Value" "PWR_FLAG" (at 190.5 50.8 90)
-      (effects (font (size 1.27 1.27)) (justify left))
-    )
-    (property "Footprint" "" (at 187.96 49.53 0)
-      (effects (font (size 1.27 1.27)) hide)
-    )
-    (property "Datasheet" "~" (at 187.96 49.53 0)
-      (effects (font (size 1.27 1.27)) hide)
-    )
-    (pin "1")
-    (instances
-      (project "THRControlModuleBoard"
-        (path "/79fd2516-dad6-414c-bb46-91ee9bfb5006"
-          (reference "#FLG02") (unit 1)
         )
       )
@@
       (effects (font (size 1.27 1.27)) hide)
     )
-    (property "Value" "GND" (at 171.45 39.37 0)
+    (property "Value" "GND" (at 171.45 40.64 0)
       (effects (font (size 1.27 1.27)))
     )
@@
       (effects (font (size 1.27 1.27)) hide)
     )
-    (property "Value" "GND" (at 196.85 48.26 0)
-      (effects (font (size 1.27 1.27)))
-    )
+    (property "Value" "GND" (at 196.85 49.53 0)
+      (effects (font (size 1.27 1.27)))
+    )

Commit message: STM32F303K8のシートを追加
Parts:
- U1: footprint Package_SO:MSOP-10-1EP_3x3mm_P0.5mm_EP1.68x1.88mm -> MSOP-10_MS
Connections:
- net CS renamed STM32F303K8/SPI__~{CS}-~{CS}
- net SCK renamed STM32F303K8/SPI__SCK-SCLK
- net SDI renamed STM32F303K8/SPI__SDI-MOSI
- net SDO renamed STM32F303K8/SPI__SDO-MISO
Other:
- added sheet STM32F303K8 (STM32F303K8.kicad_sch)
Changed lines of the file:
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@@
     (stroke (width 0) (type default))
   )
-  (wire (pts (xy 173.99 69.85) (xy 224.79 69.85))
+  (wire (pts (xy 173.99 69.85) (xy 240.03 69.85))
     (stroke (width 0) (type default))
   )
@@
     (stroke (width 0) (type default))
   )
-  (wire (pts (xy 224.79 67.31) (xy 229.87 67.31))
+  (wire (pts (xy 224.79 67.31) (xy 240.03 67.31))
     (stroke (width 0) (type default))
   )
@@
     (stroke (width 0) (type default))
   )
-  (wire (pts (xy 236.22 62.23) (xy 241.3 62.23))
+  (wire (pts (xy 236.22 62.23) (xy 240.03 62.23))
     (stroke (width 0) (type default))
   )
@@
     (stroke (width 0) (type default))
   )
-  (wire (pts (xy 231.14 64.77) (xy 234.95 64.77))
+  (wire (pts (xy 231.14 64.77) (xy 240.03 64.77))
     (stroke (width 0) (type default))
   )
@@
   (label "QMOS{slash}3-3" (at 205.74 113.03 0) (fields_autoplaced)
     (effects (font (size 1.27 1.27)) (justify left bottom))
-  )
-  (global_label "SDO" (shape output) (at 224.79 69.85 0) (fields_autoplaced)
-    (effects (font (size 1.27 1.27)) (justify left))
-    (property "Intersheetrefs" "${INTERSHEET_REFS}" (at 231.5058 69.85 0)
-      (effects (font (size 1.27 1.27)) (justify left) hide)
-    )
   )
   (global_label "Main Power Supply" (shape input) (at 232.41 137.16 0) (fields_autoplaced)
@@
     )
   )
-  (global_label "SCK" (shape input) (at 234.95 64.77 0) (fields_autoplaced)
-    (effects (font (size 1.27 1.27)) (justify left))
-    (property "Intersheetrefs" "${INTERSHEET_REFS}" (at 241.6053 64.77 0)
-      (effects (font (size 1.27 1.27)) (justify left) hide)
-    )
-  )
   (global_label "External Power Supply" (shape input) (at 38.1 114.3 180) (fields_autoplaced)
     (effects (font (size 1.27 1.27)) (justify right))
@@
     )
   )
-  (global_label "SDI" (shape input) (at 229.87 67.31 0) (fields_autoplaced)
-    (effects (font (size 1.27 1.27)) (justify left))
-    (property "Intersheetrefs" "${INTERSHEET_REFS}" (at 235.8601 67.31 0)
-      (effects (font (size 1.27 1.27)) (justify left) hide)
-    )
-  )
   (global_label "External Power Supply" (shape input) (at 85.09 120.65 180) (fields_autoplaced)
     (effects (font (size 1.27 1.27)) (justify right))
     (property "Intersheetrefs" "${INTERSHEET_REFS}" (at 60.5946 120.65 0)
       (effects (font (size 1.27 1.27)) (justify right) hide)
-    )
-  )
-  (global_label "CS" (shape bidirectional) (at 241.3 62.23 0) (fields_autoplaced)
-    (effects (font (size 1.27 1.27)) (justify left))
-    (property "Intersheetrefs" "${INTERSHEET_REFS}" (at 247.7966 62.23 0)
-      (effects (font (size 1.27 1.27)) (justify left) hide)
     )
   )
@@
       (effects (font (size 1.27 1.27)))
     )
-    (property "Footprint" "Package_SO:MSOP-10-1EP_3x3mm_P0.5mm_EP1.68x1.88mm" (at 138.43 124.46 0)
-      (effects (font (size 1.27 1.27)) (justify bottom) hide)
-    )
-    (property "Datasheet" "" (at 130.81 132.08 0)
+    (property "Footprint" "MSOP-10_MS" (at 138.43 124.46 0)
+      (effects (font (size 1.27 1.27)) (justify bottom) hide)
+    )
+    (property "Datasheet" "https://www.analog.com/media/jp/technical-documentation/data-sheets/j4416fa.pdf" (at 130.81 132.08 0)
       (effects (font (size 1.27 1.27)) hide)
     )
@@
       )
     )
+  )
+  (sheet (at 240.03 60.96) (size 29.21 10.16) (fields_autoplaced)
+    (stroke (width 0.1524) (type solid))
+    (fill (color 0 0 0 0.0000))
+    (property "Sheetname" "STM32F303K8" (at 240.03 60.2484 0)
+      (effects (font (size 1.27 1.27)) (justify left bottom))
+    )
+    (property "Sheetfile" "STM32F303K8.kicad_sch" (at 240.03 71.7046 0)
+      (effects (font (size 1.27 1.27)) (justify left top))
+    )
+    (pin "SPI__SCK-SCLK" bidirectional (at 240.03 64.77 180)
+      (effects (font (size 1.27 1.27)) (justify left))
+    )
+    (pin "SPI__~{CS}-~{CS}" passive (at 240.03 62.23 180)
+      (effects (font (size 1.27 1.27)) (justify left))
+    )
+    (pin "SPI__SDO-MISO" input (at 240.03 69.85 180)
+      (effects (font (size 1.27 1.27)) (justify left))
+    )
+    (pin "SPI__SDI-MOSI" output (at 240.03 67.31 180)
+      (effects (font (size 1.27 1.27)) (justify left))
+    )
+    (instances
+      (project "THRControlModuleBoard"
+        (path "/79fd2516-dad6-414c-bb46-91ee9bfb5006" (page "2"))
+      )
+    )

Commit message: THRControlModuleBoardを更新
Parts:
- J1, J2: footprint (none) -> CONNECTOR:CONNECTOR_2
- U1: footprint MSOP-10_MS -> Package_SO:MSOP-10_3x3mm_P0.5mm
Changed lines of the file:
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@@
       (effects (font (size 1.27 1.27)) (justify left))
     )
-    (property "Footprint" "" (at 46.99 123.19 0)
+    (property "Footprint" "CONNECTOR:CONNECTOR_2" (at 46.99 123.19 0)
       (effects (font (size 1.27 1.27)) hide)
     )
@@
       (effects (font (size 1.27 1.27)) (justify left))
     )
-    (property "Footprint" "" (at 46.99 110.49 0)
+    (property "Footprint" "CONNECTOR:CONNECTOR_2" (at 46.99 110.49 0)
       (effects (font (size 1.27 1.27)) hide)
     )
@@
       (effects (font (size 1.27 1.27)))
     )
-    (property "Footprint" "MSOP-10_MS" (at 138.43 124.46 0)
-      (effects (font (size 1.27 1.27)) (justify bottom) hide)
-    )
+    (property "Footprint" "Package_SO:MSOP-10_3x3mm_P0.5mm" (at 138.43 124.46 0)
+      (effects (font (size 1.27 1.27)) (justify bottom) hide)
+    )

Commit message: THRControlModuleBoardの更新
Parts:
- added D4, D5: LED, symbol Device:LED
- added JP1: SolderJumper_3_Open, symbol Jumper:SolderJumper_3_Open
Connections:
- net External Power Supply: now also D4.2 (A)
- net GND: now also D4.1 (K), D5.1 (K)
- net Internal Power Supply: now also D5.2 (A)
- net FAULT renamed ~{FAULT}
- net ~{FAULT}: now also JP1.1 (A)
Other:
- sheet STM32F303K8 ports: added DRDY; removed none
Changed lines of the file:
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@@
   (junction (at 220.98 137.16) (diameter 0) (color 0 0 0 0)
+  )
+  (junction (at 90.17 152.4) (diameter 0) (color 0 0 0 0)
   )
   (junction (at 204.47 67.31) (diameter 0) (color 0 0 0 0)
@@
     (stroke (width 0) (type default))
   )
+  (wire (pts (xy 99.06 161.29) (xy 99.06 162.56))
+    (stroke (width 0) (type default))
+  )
   (wire (pts (xy 38.1 123.19) (xy 41.91 123.19))
     (stroke (width 0) (type default))
@@
     (stroke (width 0) (type default))
   )
+  (wire (pts (xy 220.98 91.44) (xy 223.52 91.44))
+    (stroke (width 0) (type default))
+  )
   (wire (pts (xy 207.01 132.08) (xy 207.01 129.54))
     (stroke (width 0) (type default))
@@
     (stroke (width 0) (type default))
   )
+  (wire (pts (xy 90.17 161.29) (xy 90.17 152.4))
+    (stroke (width 0) (type default))
+  )
   (wire (pts (xy 39.37 114.3) (xy 39.37 113.03))
     (stroke (width 0) (type default))
@@
     (stroke (width 0) (type default))
   )
+  (wire (pts (xy 90.17 152.4) (xy 189.23 152.4))
+    (stroke (width 0) (type default))
+  )
   (wire (pts (xy 218.44 152.4) (xy 218.44 137.16))
     (stroke (width 0) (type default))
@@
     (stroke (width 0) (type default))
   )
+  (wire (pts (xy 90.17 111.76) (xy 90.17 120.65))
+    (stroke (width 0) (type default))
+  )
   (wire (pts (xy 175.26 77.47) (xy 175.26 78.74))
     (stroke (width 0) (type default))
   )
-  (wire (pts (xy 85.09 152.4) (xy 189.23 152.4))
+  (wire (pts (xy 85.09 152.4) (xy 90.17 152.4))
     (stroke (width 0) (type default))
   )
@@
     (stroke (width 0) (type default))
   )
+  (wire (pts (xy 91.44 111.76) (xy 90.17 111.76))
+    (stroke (width 0) (type default))
+  )
   (wire (pts (xy 130.81 57.15) (xy 130.81 62.23))
     (stroke (width 0) (type default))
@@
     (stroke (width 0) (type default))
   )
+  (wire (pts (xy 223.52 91.44) (xy 223.52 88.9))
+    (stroke (width 0) (type default))
+  )
   (wire (pts (xy 104.14 57.15) (xy 106.68 57.15))
     (stroke (width 0) (type default))
@@
     (stroke (width 0) (type default))
   )
+  (wire (pts (xy 97.79 161.29) (xy 99.06 161.29))
+    (stroke (width 0) (type default))
+  )
   (wire (pts (xy 214.63 129.54) (xy 214.63 128.27))
     (stroke (width 0) (type default))
@@
     (stroke (width 0) (type default))
   )
+  (wire (pts (xy 100.33 111.76) (xy 100.33 113.03))
+    (stroke (width 0) (type default))
+  )
   (wire (pts (xy 186.69 134.62) (xy 189.23 134.62))
     (stroke (width 0) (type default))
@@
     (stroke (width 0) (type default))
   )
+  (wire (pts (xy 99.06 111.76) (xy 100.33 111.76))
+    (stroke (width 0) (type default))
+  )
   (wire (pts (xy 41.91 125.73) (xy 39.37 125.73))
     (stroke (width 0) (type default))
   )
   (wire (pts (xy 209.55 40.64) (xy 209.55 44.45))
+    (stroke (width 0) (type default))
+  )
+  (wire (pts (xy 236.22 72.39) (xy 240.03 72.39))
     (stroke (width 0) (type default))
   )
@@
     )
   )
-  (global_label "FAULT" (shape output) (at 175.26 57.15 0) (fields_autoplaced)
+  (global_label "~{FAULT}" (shape output) (at 175.26 57.15 0) (fields_autoplaced)
     (effects (font (face "KiCad Font") (size 1.27 1.27)) (justify left))
     (property "Intersheetrefs" "${INTERSHEET_REFS}" (at 183.6692 57.15 0)
@@
     )
   )
+  (global_label "~{FAULT}" (shape input) (at 220.98 91.44 180) (fields_autoplaced)
+    (effects (font (size 1.27 1.27)) (justify right))
+    (property "Intersheetrefs" "${INTERSHEET_REFS}" (at 212.5708 91.44 0)
+      (effects (font (size 1.27 1.27)) (justify right) hide)
+    )
+  )
   (global_label "External Power Supply" (shape input) (at 38.1 114.3 180) (fields_autoplaced)
     (effects (font (size 1.27 1.27)) (justify right))
@@
     )
   )
+  (global_label "DRDY" (shape output) (at 236.22 72.39 180) (fields_autoplaced)
+    (effects (font (face "KiCad Font") (size 1.27 1.27)) (justify right))
+    (property "Intersheetrefs" "${INTERSHEET_REFS}" (at 228.4156 72.39 0)
+      (effects (font (size 1.27 1.27)) (justify right) hide)
+    )
+  )
   (symbol (lib_id "Device:D") (at 220.98 67.31 180) (unit 1)
     (in_bom yes) (on_board yes) (dnp no) (fields_autoplaced)
@@
         (path "/79fd2516-dad6-414c-bb46-91ee9bfb5006"
           (reference "C4") (unit 1)
+        )
+      )
+    )
+  )
+  (symbol (lib_id "Device:LED") (at 95.25 111.76 180) (unit 1)
+    (in_bom yes) (on_board yes) (dnp no) (fields_autoplaced)
+    (property "Reference" "D4" (at 96.8375 105.41 0)
+      (effects (font (size 1.27 1.27)))
+    )
+    (property "Value" "LED" (at 96.8375 107.95 0)
+      (effects (font (size 1.27 1.27)))
+    )
+    (property "Footprint" "" (at 95.25 111.76 0)
+      (effects (font (size 1.27 1.27)) hide)
+    )
+    (property "Datasheet" "~" (at 95.25 111.76 0)
+      (effects (font (size 1.27 1.27)) hide)
+    )
+    (pin "1")
+    (pin "2")
+    (instances
+      (project "THRControlModuleBoard"
+        (path "/79fd2516-dad6-414c-bb46-91ee9bfb5006"
+          (reference "D4") (unit 1)
+        )
+      )
+    )
+  )
+  (symbol (lib_id "Jumper:SolderJumper_3_Open") (at 223.52 83.82 90) (unit 1)
+    (in_bom yes) (on_board yes) (dnp no) (fields_autoplaced)
+    (property "Reference" "JP1" (at 220.98 83.185 90)
+      (effects (font (size 1.27 1.27)) (justify left))
+    )
+    (property "Value" "SolderJumper_3_Open" (at 220.98 85.725 90)
+      (effects (font (size 1.27 1.27)) (justify left))
+    )
+    (property "Footprint" "" (at 223.52 83.82 0)
+      (effects (font (size 1.27 1.27)) hide)
+    )
+    (property "Datasheet" "~" (at 223.52 83.82 0)
+      (effects (font (size 1.27 1.27)) hide)
+    )
+    (pin "1")
+    (pin "2")
+    (pin "3")
+    (instances
+      (project "THRControlModuleBoard"
+        (path "/79fd2516-dad6-414c-bb46-91ee9bfb5006"
+          (reference "JP1") (unit 1)
         )
       )
@@
         (path "/79fd2516-dad6-414c-bb46-91ee9bfb5006"
           (reference "#FLG01") (unit 1)
+        )
+      )
+    )
+  )
+  (symbol (lib_id "power:GND") (at 100.33 113.03 0) (unit 1)
+    (in_bom yes) (on_board yes) (dnp no) (fields_autoplaced)
+    (property "Reference" "#PWR019" (at 100.33 119.38 0)
+      (effects (font (size 1.27 1.27)) hide)
+    )
+    (property "Value" "GND" (at 100.33 118.11 0)
+      (effects (font (size 1.27 1.27)))
+    )
+    (property "Footprint" "" (at 100.33 113.03 0)
+      (effects (font (size 1.27 1.27)) hide)
+    )
+    (property "Datasheet" "" (at 100.33 113.03 0)
+      (effects (font (size 1.27 1.27)) hide)
+    )
+    (pin "1")
+    (instances
+      (project "THRControlModuleBoard"
+        (path "/79fd2516-dad6-414c-bb46-91ee9bfb5006"
+          (reference "#PWR019") (unit 1)
+        )
+      )
+    )
+  )
+  (symbol (lib_id "power:GND") (at 99.06 162.56 0) (unit 1)
+    (in_bom yes) (on_board yes) (dnp no) (fields_autoplaced)
+    (property "Reference" "#PWR03" (at 99.06 168.91 0)
+      (effects (font (size 1.27 1.27)) hide)
+    )
+    (property "Value" "GND" (at 99.06 167.64 0)
+      (effects (font (size 1.27 1.27)))
+    )
+    (property "Footprint" "" (at 99.06 162.56 0)
+      (effects (font (size 1.27 1.27)) hide)
+    )
+    (property "Datasheet" "" (at 99.06 162.56 0)
+      (effects (font (size 1.27 1.27)) hide)
+    )
+    (pin "1")
+    (instances
+      (project "THRControlModuleBoard"
+        (path "/79fd2516-dad6-414c-bb46-91ee9bfb5006"
+          (reference "#PWR03") (unit 1)
         )
       )
@@
         (path "/79fd2516-dad6-414c-bb46-91ee9bfb5006"
           (reference "J1") (unit 1)
+        )
+      )
+    )
+  )
+  (symbol (lib_id "Device:LED") (at 93.98 161.29 180) (unit 1)
+    (in_bom yes) (on_board yes) (dnp no) (fields_autoplaced)
+    (property "Reference" "D5" (at 95.5675 154.94 0)
+      (effects (font (size 1.27 1.27)))
+    )
+    (property "Value" "LED" (at 95.5675 157.48 0)
+      (effects (font (size 1.27 1.27)))
+    )
+    (property "Footprint" "" (at 93.98 161.29 0)
+      (effects (font (size 1.27 1.27)) hide)
+    )
+    (property "Datasheet" "~" (at 93.98 161.29 0)
+      (effects (font (size 1.27 1.27)) hide)
+    )
+    (pin "1")
+    (pin "2")
+    (instances
+      (project "THRControlModuleBoard"
+        (path "/79fd2516-dad6-414c-bb46-91ee9bfb5006"
+          (reference "D5") (unit 1)
         )
       )
@@
     )
   )
-  (sheet (at 240.03 60.96) (size 29.21 10.16) (fields_autoplaced)
+  (sheet (at 240.03 59.69) (size 30.48 15.24) (fields_autoplaced)
     (stroke (width 0.1524) (type solid))
     (fill (color 0 0 0 0.0000))
-    (property "Sheetname" "STM32F303K8" (at 240.03 60.2484 0)
+    (property "Sheetname" "STM32F303K8" (at 240.03 58.9784 0)
       (effects (font (size 1.27 1.27)) (justify left bottom))
     )
-    (property "Sheetfile" "STM32F303K8.kicad_sch" (at 240.03 71.7046 0)
+    (property "Sheetfile" "STM32F303K8.kicad_sch" (at 240.03 75.5146 0)
       (effects (font (size 1.27 1.27)) (justify left top))
     )
@@
       (effects (font (size 1.27 1.27)) (justify left))
     )
+    (pin "DRDY" input (at 240.03 72.39 180)
+      (effects (font (size 1.27 1.27)) (justify left))
+    )

Commit message: THRControlModuleBoardにRS485系統を追加しました。
Parts:
- J1, J2: footprint CONNECTOR:CONNECTOR_2 -> CONNECTOR:CONNECTOR_2-STRAIGHT
Changed lines of the file:
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@@
       (effects (font (size 1.27 1.27)) (justify left))
     )
-    (property "Footprint" "CONNECTOR:CONNECTOR_2" (at 46.99 123.19 0)
+    (property "Footprint" "CONNECTOR:CONNECTOR_2-STRAIGHT" (at 46.99 123.19 0)
       (effects (font (size 1.27 1.27)) hide)
     )
@@
       (effects (font (size 1.27 1.27)) (justify left))
     )
-    (property "Footprint" "CONNECTOR:CONNECTOR_2" (at 46.99 110.49 0)
-      (effects (font (size 1.27 1.27)) hide)
-    )
+    (property "Footprint" "CONNECTOR:CONNECTOR_2-STRAIGHT" (at 46.99 110.49 0)
+      (effects (font (size 1.27 1.27)) hide)
+    )

Commit message: THRControlModuleBoardの更新
Parts:
- added R10: 1k, LED_SMD:LED_0805_2012Metric_Pad1.15x1.40mm_HandSolder, symbol Device:R
- added R9: 1K, LED_SMD:LED_0805_2012Metric_Pad1.15x1.40mm_HandSolder, symbol Device:R
- C1, C2: footprint Capacitor_SMD:C_0603_1608Metric_Pad1.08x0.95mm_HandSolder -> Capacitor_SMD:C_0805_2012Metric_Pad1.18x1.45mm_HandSolder
- D4, D5: footprint (none) -> LED_SMD:LED_0805_2012Metric_Pad1.15x1.40mm_HandSolder
- R1, R2, R3: footprint Resistor_SMD:R_0603_1608Metric_Pad0.98x0.95mm_HandSolder -> Resistor_SMD:R_0805_2012Metric_Pad1.20x1.40mm_HandSolder
Connections:
- net External Power Supply: now also R10.1; no longer D4.2 (A)
- net Internal Power Supply: no longer D5.2 (A)
- net at Q3.1 (G), U1.6 (G2): now also R9.2
- new net: D4.2 (A), R10.2
- new net: D5.2 (A), R9.1
Other:
- moved on the sheet: C2, D4, D5, Q2
