File: Projects/KiCad/THRControlModuleBoard/THRControlModuleBoard.kicad_sch (KiCad schematic)
At the start: 31 parts, among them J1 Conn_01x02_Socket, J2 Conn_01x02_Socket, J3 Screw_Terminal_01x02, Q1 Q_PMOS_GDS, Q2 Q_PMOS_GDS, Q3 Q_PMOS_GDS, U1 LTC4416EMS#PBF, U2 MAX31856MUD+T

Commit message: THRControlModuleを更新
Parts:
- removed J3: Screw_Terminal_01x02, TerminalBlock:TerminalBlock_Altech_AK300-2_P5.00mm, symbol Connector:Screw_Terminal_01x02
- added J6: PCC-SMP-K-5, OMEGA_PCC-SMP-K-5, symbol PCC-SMP-K-5:PCC-SMP-K-5
Connections:
- net BIAS: now also J6.N (NEG)
- net GND: now also J6.S1 (SHIELD), J6.S2 (SHIELD)
- net at R5.1: now also J6.P (POS)
Changed lines of the file:
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@@
+    (stroke (width 0) (type default))
+  )
+  (wire (pts (xy 87.63 62.23) (xy 88.9 62.23))
     (stroke (width 0) (type default))
   )
@@
     (stroke (width 0) (type default))
   )
-  (wire (pts (xy 104.14 54.61) (xy 106.68 54.61))
+  (wire (pts (xy 87.63 54.61) (xy 106.68 54.61))
     (stroke (width 0) (type default))
   )
@@
     (stroke (width 0) (type default))
   )
+  (wire (pts (xy 88.9 62.23) (xy 88.9 63.5))
+    (stroke (width 0) (type default))
+  )
   (wire (pts (xy 121.92 49.53) (xy 121.92 52.07))
     (stroke (width 0) (type default))
@@
     (stroke (width 0) (type default))
   )
-  (wire (pts (xy 104.14 57.15) (xy 106.68 57.15))
+  (wire (pts (xy 87.63 57.15) (xy 106.68 57.15))
     (stroke (width 0) (type default))
   )
@@
     )
   )
+  (symbol (lib_id "PCC-SMP-K-5:PCC-SMP-K-5") (at 77.47 57.15 0) (unit 1)
+    (in_bom yes) (on_board yes) (dnp no) (fields_autoplaced)
+    (property "Reference" "J6" (at 77.47 48.26 0)
+      (effects (font (size 1.27 1.27)))
+    )
+    (property "Value" "PCC-SMP-K-5" (at 77.47 50.8 0)
+      (effects (font (size 1.27 1.27)))
+    )
+    (property "Footprint" "OMEGA_PCC-SMP-K-5" (at 77.47 57.15 0)
+      (effects (font (size 1.27 1.27)) (justify bottom) hide)
+    )
+    (property "Datasheet" "" (at 77.47 57.15 0)
+      (effects (font (size 1.27 1.27)) hide)
+    )
+    (property "MANUFACTURER" "OMEGA" (at 77.47 57.15 0)
+      (effects (font (size 1.27 1.27)) (justify bottom) hide)
+    )
+    (property "PARTREV" "N/A" (at 77.47 57.15 0)
+      (effects (font (size 1.27 1.27)) (justify bottom) hide)
+    )
+    (property "STANDARD" "Manufacturer Recommendations" (at 77.47 57.15 0)
+      (effects (font (size 1.27 1.27)) (justify bottom) hide)
+    )
+    (property "MAXIMUM_PACKAGE_HEIGHT" "6.3 mm" (at 77.47 57.15 0)
+      (effects (font (size 1.27 1.27)) (justify bottom) hide)
+    )
+    (pin "N")
+    (pin "P")
+    (pin "S1")
+    (pin "S2")
+    (instances
+      (project "THRControlModuleBoard"
+        (path "/79fd2516-dad6-414c-bb46-91ee9bfb5006"
+          (reference "J6") (unit 1)
+        )
+      )
+    )
+  )
   (symbol (lib_id "power:+3.3V") (at 204.47 43.18 0) (unit 1)
     (in_bom yes) (on_board yes) (dnp no) (fields_autoplaced)
@@
         (path "/79fd2516-dad6-414c-bb46-91ee9bfb5006"
           (reference "#PWR010") (unit 1)
+        )
+      )
+    )
+  )
+  (symbol (lib_id "power:GND") (at 88.9 63.5 0) (unit 1)
+    (in_bom yes) (on_board yes) (dnp no) (fields_autoplaced)
+    (property "Reference" "#PWR030" (at 88.9 69.85 0)
+      (effects (font (size 1.27 1.27)) hide)
+    )
+    (property "Value" "GND" (at 88.9 68.58 0)
+      (effects (font (size 1.27 1.27)))
+    )
+    (property "Footprint" "" (at 88.9 63.5 0)
+      (effects (font (size 1.27 1.27)) hide)
+    )
+    (property "Datasheet" "" (at 88.9 63.5 0)
+      (effects (font (size 1.27 1.27)) hide)
+    )
+    (pin "1")
+    (instances
+      (project "THRControlModuleBoard"
+        (path "/79fd2516-dad6-414c-bb46-91ee9bfb5006"
+          (reference "#PWR030") (unit 1)
         )
       )
@@
         )
       )
-    )
-  )
-  (symbol (lib_id "Connector:Screw_Terminal_01x02") (at 99.06 57.15 180) (unit 1)
-    (in_bom yes) (on_board yes) (dnp no)
-    (property "Reference" "J3" (at 99.06 48.26 0)
-      (effects (font (size 1.27 1.27)))
-    )
-    (property "Value" "Screw_Terminal_01x02" (at 99.06 50.8 0)
-      (effects (font (size 1.27 1.27)))
-    )
-    (property "Footprint" "TerminalBlock:TerminalBlock_Altech_AK300-2_P5.00mm" (at 99.06 57.15 0)
-      (effects (font (size 1.27 1.27)) hide)
-    )
-    (property "Datasheet" "~" (at 99.06 57.15 0)
-      (effects (font (size 1.27 1.27)) hide)
-    )
-    (pin "1")
-    (pin "2")
-    (instances
-      (project "THRControlModuleBoard"
-        (path "/79fd2516-dad6-414c-bb46-91ee9bfb5006"
-          (reference "J3") (unit 1)
-        )
-      )

Commit message: THRControlModuleを更新
Parts:
- added J3: Screw_Terminal_01x02, TerminalBlock:TerminalBlock_Altech_AK300-2_P5.00mm, symbol Connector:Screw_Terminal_01x02
Connections:
- net BIAS: now also J3.1 (Pin_1)
- net at J6.P (POS), R5.1: now also J3.2 (Pin_2)
Changed lines of the file:
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@@
 (kicad_sch (version 20230121) (generator eeschema)
   (paper "A4")
+  (junction (at 97.79 57.15) (diameter 0) (color 0 0 0 0)
+  )
   (junction (at 228.6 137.16) (diameter 0) (color 0 0 0 0)
   )
@@
   )
   (junction (at 182.88 26.67) (diameter 0) (color 0 0 0 0)
+  )
+  (junction (at 101.6 54.61) (diameter 0) (color 0 0 0 0)
   )
   (junction (at 120.65 139.7) (diameter 0) (color 0 0 0 0)
@@
   (no_connect (at 130.81 139.7))
   (no_connect (at 130.81 142.24))
+  (wire (pts (xy 101.6 54.61) (xy 106.68 54.61))
+    (stroke (width 0) (type default))
+  )
   (wire (pts (xy 212.09 157.48) (xy 212.09 142.24))
     (stroke (width 0) (type default))
@@
     (stroke (width 0) (type default))
   )
+  (wire (pts (xy 96.52 43.18) (xy 97.79 43.18))
+    (stroke (width 0) (type default))
+  )
   (wire (pts (xy 102.87 134.62) (xy 102.87 132.08))
     (stroke (width 0) (type default))
@@
     (stroke (width 0) (type default))
   )
+  (wire (pts (xy 96.52 40.64) (xy 101.6 40.64))
+    (stroke (width 0) (type default))
+  )
   (wire (pts (xy 90.17 123.19) (xy 90.17 120.65))
     (stroke (width 0) (type default))
   )
+  (wire (pts (xy 101.6 40.64) (xy 101.6 54.61))
+    (stroke (width 0) (type default))
+  )
   (wire (pts (xy 121.92 62.23) (xy 121.92 64.77))
     (stroke (width 0) (type default))
   )
-  (wire (pts (xy 87.63 54.61) (xy 106.68 54.61))
+  (wire (pts (xy 87.63 54.61) (xy 101.6 54.61))
     (stroke (width 0) (type default))
   )
@@
     (stroke (width 0) (type default))
   )
+  (wire (pts (xy 97.79 57.15) (xy 106.68 57.15))
+    (stroke (width 0) (type default))
+  )
   (wire (pts (xy 130.81 57.15) (xy 130.81 62.23))
     (stroke (width 0) (type default))
@@
     (stroke (width 0) (type default))
   )
-  (wire (pts (xy 87.63 57.15) (xy 106.68 57.15))
+  (wire (pts (xy 87.63 57.15) (xy 97.79 57.15))
     (stroke (width 0) (type default))
   )
@@
   )
   (wire (pts (xy 195.58 43.18) (xy 196.85 43.18))
+    (stroke (width 0) (type default))
+  )
+  (wire (pts (xy 97.79 43.18) (xy 97.79 57.15))
     (stroke (width 0) (type default))
   )
@@
         )
       )
+    )
+  )
+  (symbol (lib_id "Connector:Screw_Terminal_01x02") (at 91.44 43.18 180) (unit 1)
+    (in_bom yes) (on_board yes) (dnp no) (fields_autoplaced)
+    (property "Reference" "J3" (at 91.44 35.56 0)
+      (effects (font (size 1.27 1.27)))
+    )
+    (property "Value" "Screw_Terminal_01x02" (at 91.44 38.1 0)
+      (effects (font (size 1.27 1.27)))
+    )
+    (property "Footprint" "TerminalBlock:TerminalBlock_Altech_AK300-2_P5.00mm" (at 91.44 43.18 0)
+      (effects (font (size 1.27 1.27)) hide)
+    )
+    (property "Datasheet" "~" (at 91.44 43.18 0)
+      (effects (font (size 1.27 1.27)) hide)
+    )
+    (pin "1")
+    (pin "2")
+    (instances
+      (project "THRControlModuleBoard"
+        (path "/79fd2516-dad6-414c-bb46-91ee9bfb5006"
+          (reference "J3") (unit 1)
+        )
+      )

Commit message: 取付穴位置等を追加
Parts:
- added H1, H2, H3, H4: MountingHole, MountingHole:MountingHole_4.5mm, symbol Mechanical:MountingHole
Changed lines of the file:
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@@
+    )
+  )
+  (symbol (lib_id "Mechanical:MountingHole") (at 40.64 45.72 0) (unit 1)
+    (in_bom yes) (on_board yes) (dnp no) (fields_autoplaced)
+    (property "Reference" "H2" (at 43.18 45.085 0)
+      (effects (font (size 1.27 1.27)) (justify left))
+    )
+    (property "Value" "MountingHole" (at 43.18 47.625 0)
+      (effects (font (size 1.27 1.27)) (justify left))
+    )
+    (property "Footprint" "MountingHole:MountingHole_4.5mm" (at 40.64 45.72 0)
+      (effects (font (size 1.27 1.27)) hide)
+    )
+    (property "Datasheet" "~" (at 40.64 45.72 0)
+      (effects (font (size 1.27 1.27)) hide)
+    )
+    (instances
+      (project "THRControlModuleBoard"
+        (path "/79fd2516-dad6-414c-bb46-91ee9bfb5006"
+          (reference "H2") (unit 1)
+        )
+      )
     )
   )
@@
         (path "/79fd2516-dad6-414c-bb46-91ee9bfb5006"
           (reference "#PWR09") (unit 1)
+        )
+      )
+    )
+  )
+  (symbol (lib_id "Mechanical:MountingHole") (at 40.64 39.37 0) (unit 1)
+    (in_bom yes) (on_board yes) (dnp no) (fields_autoplaced)
+    (property "Reference" "H1" (at 43.18 38.735 0)
+      (effects (font (size 1.27 1.27)) (justify left))
+    )
+    (property "Value" "MountingHole" (at 43.18 41.275 0)
+      (effects (font (size 1.27 1.27)) (justify left))
+    )
+    (property "Footprint" "MountingHole:MountingHole_4.5mm" (at 40.64 39.37 0)
+      (effects (font (size 1.27 1.27)) hide)
+    )
+    (property "Datasheet" "~" (at 40.64 39.37 0)
+      (effects (font (size 1.27 1.27)) hide)
+    )
+    (instances
+      (project "THRControlModuleBoard"
+        (path "/79fd2516-dad6-414c-bb46-91ee9bfb5006"
+          (reference "H1") (unit 1)
         )
       )
@@
     )
   )
+  (symbol (lib_id "Mechanical:MountingHole") (at 40.64 58.42 0) (unit 1)
+    (in_bom yes) (on_board yes) (dnp no) (fields_autoplaced)
+    (property "Reference" "H4" (at 43.18 57.785 0)
+      (effects (font (size 1.27 1.27)) (justify left))
+    )
+    (property "Value" "MountingHole" (at 43.18 60.325 0)
+      (effects (font (size 1.27 1.27)) (justify left))
+    )
+    (property "Footprint" "MountingHole:MountingHole_4.5mm" (at 40.64 58.42 0)
+      (effects (font (size 1.27 1.27)) hide)
+    )
+    (property "Datasheet" "~" (at 40.64 58.42 0)
+      (effects (font (size 1.27 1.27)) hide)
+    )
+    (instances
+      (project "THRControlModuleBoard"
+        (path "/79fd2516-dad6-414c-bb46-91ee9bfb5006"
+          (reference "H4") (unit 1)
+        )
+      )
+    )
+  )
   (symbol (lib_id "Device:Q_PMOS_GDS") (at 199.39 123.19 90) (unit 1)
     (in_bom yes) (on_board yes) (dnp no) (fields_autoplaced)
@@
         )
       )
+    )
+  )
+  (symbol (lib_id "Mechanical:MountingHole") (at 40.64 52.07 0) (unit 1)
+    (in_bom yes) (on_board yes) (dnp no) (fields_autoplaced)
+    (property "Reference" "H3" (at 43.18 51.435 0)
+      (effects (font (size 1.27 1.27)) (justify left))
+    )
+    (property "Value" "MountingHole" (at 43.18 53.975 0)
+      (effects (font (size 1.27 1.27)) (justify left))
+    )
+    (property "Footprint" "MountingHole:MountingHole_4.5mm" (at 40.64 52.07 0)
+      (effects (font (size 1.27 1.27)) hide)
+    )
+    (property "Datasheet" "~" (at 40.64 52.07 0)
+      (effects (font (size 1.27 1.27)) hide)
+    )
+    (instances
+      (project "THRControlModuleBoard"
+        (path "/79fd2516-dad6-414c-bb46-91ee9bfb5006"
+          (reference "H3") (unit 1)
+        )
+      )

Commit message: KiCADを更新
Parts:
- removed JP1: SolderJumper_3_Open, symbol Jumper:SolderJumper_3_Open
- added JP1, JP2: SolderJumper_2_Bridged, Jumper:SolderJumper-2_P1.3mm_Open_TrianglePad1.0x1.5mm, symbol Jumper:SolderJumper_2_Bridged
Connections:
- net DRDY: now also JP2.1 (A)
- net ~{FAULT}: now also JP1.1 (A)
- net +3.3V renamed NanoEvery_3.3V
- net STM32F303K8/SPI__SCK-SCLK renamed NanoEvery/MAX31856__SCK-SCLK
- net STM32F303K8/SPI__SDI-MOSI renamed NanoEvery/MAX31856__SDI-MOSI
- net STM32F303K8/SPI__SDO-MISO renamed NanoEvery/MAX31856__SDO-MISO
- net STM32F303K8/SPI__~{CS}-~{CS} renamed NanoEvery/MAX31856__~{CS}-~{CS}
- new net NanoEvery/MAX31856__DRDY-DRDY: JP2.2 (B)
- new net NanoEvery/MAX31856__FAULT-FAULT: JP1.2 (B)
Other:
- removed sheet STM32F303K8
- added sheet NanoEvery (NanoEvery.kicad_sch)

Commit message: KiCADを更新
Parts:
- added JP3, JP4, JP5, JP6: SolderJumper_2_Bridged, Jumper:SolderJumper-2_P1.3mm_Open_TrianglePad1.0x1.5mm, symbol Jumper:SolderJumper_2_Bridged
Connections:
- net NanoEvery/MAX31856__~{CS}-~{CS}: now also JP6.2 (B); no longer D1.1 (K)
- net NanoEvery/MAX31856__SCK-SCLK: no longer names the net of D2.1 (K)
- net NanoEvery/MAX31856__SCK-SCLK: now also JP5.1 (A)
- net NanoEvery/MAX31856__SDI-MOSI: no longer names the net of D3.1 (K)
- net NanoEvery/MAX31856__SDI-MOSI: now also JP4.1 (A)
- net NanoEvery/MAX31856__SDO-MISO: no longer names the net of U2.11 (SDO)
- net NanoEvery/MAX31856__SDO-MISO: now also JP3.1 (A)
- new net: D1.1 (K), JP6.1 (A)
- new net NanoEvery/SPI__SCK-SCLK: JP5.2 (B)
- new net NanoEvery/SPI__SDI-MOSI: JP4.2 (B)
- new net NanoEvery/SPI__SDO-MISO: JP3.2 (B)
Other:
- sheet NanoEvery ports: added SPI__SCK-SCLK, SPI__SDI-MOSI, SPI__SDO-MISO; removed MAX31856__SCK-SCLK, MAX31856__SDI-MOSI, MAX31856__SDO-MISO
- moved on the sheet: D1, D2, D3, JP1, JP2

Commit message: MAX31855、CAN、一部コネクタの追加。 基板形状は供給待ち。
Parts:
- renumbered C6 to C2, C5 to C3, C7 to C4, C3 to C5, C4 to C6, C2 to C7, D4 to D1, D3 to D2, D2 to D3, D1 to D4, J6 to J3, J3 to J4, JP2 to JP1, JP1 to JP2, JP6 to JP3, JP5 to JP4, JP4 to JP5, JP3 to JP6, Q3 to Q2, Q2 to Q3, R10 to R1, R9 to R10, R5 to R3, R3 to R5, R1 to R6, R8 to R7, R7 to R8, R6 to R9
Connections:
- net NanoEvery/SPI__SCK-SCLK renamed NanoEvery/SPI__SCLK
- net NanoEvery/SPI__SDI-MOSI renamed NanoEvery/SPI__MOSI
- net NanoEvery/SPI__SDO-MISO renamed NanoEvery/SPI__MISO
- net NanoEvery_3.3V renamed +3.3V
Other:
- sheet NanoEvery ports: added SPI__MISO, SPI__MOSI, SPI__SCLK; removed NanoEvery_3.3V, SPI__SCK-SCLK, SPI__SDI-MOSI, SPI__SDO-MISO

Commit message: PCBにQRコードを追加
Parts:
- C1: value 2u -> 2μF
- C7: value 4.7u -> 4.7μF
Changed lines of the file:
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@@
       (effects (font (size 1.27 1.27)) (justify left))
     )
-    (property "Value" "4.7u" (at 232.41 142.875 0)
+    (property "Value" "4.7μF" (at 232.41 142.875 0)
       (effects (font (size 1.27 1.27)) (justify left))
     )
@@
       (effects (font (size 1.27 1.27)) (justify left))
     )
-    (property "Value" "2u" (at 93.98 128.905 0)
-      (effects (font (size 1.27 1.27)) (justify left))
-    )
+    (property "Value" "2μF" (at 93.98 128.905 0)
+      (effects (font (size 1.27 1.27)) (justify left))
+    )

Commit message: 外形を大方決めた
Parts:
- removed C1: 2μF, Capacitor_SMD:C_0805_2012Metric_Pad1.18x1.45mm_HandSolder, symbol Device:C
- removed C7: 4.7μF, Capacitor_SMD:C_0805_2012Metric_Pad1.18x1.45mm_HandSolder, symbol Device:C
- removed D1, D5: LED, LED_SMD:LED_0805_2012Metric_Pad1.15x1.40mm_HandSolder, symbol Device:LED
- removed J1, J2: Conn_01x02_Socket, CONNECTOR:CONNECTOR_2-STRAIGHT, symbol Connector:Conn_01x02_Socket
- removed JP3, JP4, JP5, JP6: SolderJumper_2_Bridged, Jumper:SolderJumper-2_P1.3mm_Open_TrianglePad1.0x1.5mm, symbol Jumper:SolderJumper_2_Bridged
- removed Q1, Q2, Q3: Q_PMOS_GDS, Package_TO_SOT_SMD:ATPAK-2, symbol Device:Q_PMOS_GDS
- removed R1: 1k, LED_SMD:LED_0805_2012Metric_Pad1.15x1.40mm_HandSolder, symbol Device:R
- removed R10: 1K, LED_SMD:LED_0805_2012Metric_Pad1.15x1.40mm_HandSolder, symbol Device:R
- removed R2: 10k, Resistor_SMD:R_0805_2012Metric_Pad1.20x1.40mm_HandSolder, symbol Device:R
- removed R5: 120k, Resistor_SMD:R_0805_2012Metric_Pad1.20x1.40mm_HandSolder, symbol Device:R
- removed R6: 68k, Resistor_SMD:R_0805_2012Metric_Pad1.20x1.40mm_HandSolder, symbol Device:R
- removed U1: LTC4416EMS#PBF, Package_SO:MSOP-10_3x3mm_P0.5mm, symbol LTC4416EMS_PBF:LTC4416EMS#PBF
- added J5, J6: Conn_02x03_Odd_Even, Connector_PinHeader_2.00mm:PinHeader_2x03_P2.00mm_Vertical, symbol Connector_Generic:Conn_02x03_Odd_Even
- C1: renamed from C2; footprint Capacitor_SMD:C_0805_2012Metric_Pad1.18x1.45mm_HandSolder -> Capacitor_SMD:C_0603_1608Metric_Pad1.08x0.95mm_HandSolder
- C2: renamed from C3; footprint Capacitor_SMD:C_0805_2012Metric_Pad1.18x1.45mm_HandSolder -> Capacitor_SMD:C_0603_1608Metric_Pad1.08x0.95mm_HandSolder
- C3: renamed from C4; footprint Capacitor_SMD:C_0805_2012Metric_Pad1.18x1.45mm_HandSolder -> Capacitor_SMD:C_0603_1608Metric_Pad1.08x0.95mm_HandSolder
- C4: renamed from C5; footprint Capacitor_SMD:C_0805_2012Metric_Pad1.18x1.45mm_HandSolder -> Capacitor_SMD:C_0603_1608Metric_Pad1.08x0.95mm_HandSolder
- C5: renamed from C6; footprint Capacitor_SMD:C_0805_2012Metric_Pad1.18x1.45mm_HandSolder -> Capacitor_SMD:C_0603_1608Metric_Pad1.08x0.95mm_HandSolder
- D1: renamed from D2; footprint Diode_SMD:D_0805_2012Metric_Pad1.15x1.40mm_HandSolder -> Diode_SMD:D_SOD-123
- D2: renamed from D3; footprint Diode_SMD:D_0805_2012Metric_Pad1.15x1.40mm_HandSolder -> Diode_SMD:D_SOD-123
- D3: renamed from D4; footprint Diode_SMD:D_0805_2012Metric_Pad1.15x1.40mm_HandSolder -> Diode_SMD:D_SOD-123
- J1: renamed from J3; footprint OMEGA_PCC-SMP-K-5 -> PCC-SMP-K-5:OMEGA_PCC-SMP-K-5
- J2: renamed from J4; footprint TerminalBlock:TerminalBlock_Altech_AK300-2_P5.00mm -> MAX31856MUD_T:RS_PRO_611-8157
- U1: renamed from U2; footprint Package_SO:TSSOP-14_4.4x5mm_P0.65mm -> MAX31856MUD_T:SOP65P640X110-14N
- renumbered R3 to R1, R4 to R2, R7 to R3, R8 to R4, R9 to R5
Connections:
- net GND: now also J5.1 (Pin_1), J5.3 (Pin_3), J6.1 (Pin_1)
- net NanoEvery/MAX31856__~{CS}-~{CS}: now also D3.1 (K)
- net NanoEvery/SPI__MISO: now also U1.11 (SDO)
- net NanoEvery/SPI__MOSI: now also D1.1 (K)
- net NanoEvery/SPI__SCLK: now also D2.1 (K)
- new net +12V: J5.2 (Pin_2)
- new net +VDC: J5.4 (Pin_4), J6.6 (Pin_6)
- new net CAN__H: J5.6 (Pin_6)
- new net CAN__L: J5.5 (Pin_5)
- new net RS405_Servo__Closeinput: J6.5 (Pin_5)
- new net RS405_Servo__Openinput: J6.3 (Pin_3)
- new net Umbilical__launchInput: J6.4 (Pin_4)
- new net Umbilical__waitingInput: J6.2 (Pin_2)
- no-connect marks 2 -> 0
Other:
- sheet NanoEvery ports: added CAN__H, CAN__L, Umbilical__launchInput, Umbilical__waitingInput; removed none
- moved on the sheet: C4, C5, D1, D2, D3, R3, R4, R5
