File: Projects/KiCad/THRControlModuleBoard/NanoEvery.kicad_sch (KiCad schematic)
At the start: 44 parts, among them IC1 LTC1480CN8#PBF, IC2 LTC1480CN8#PBF, J4 Conn_01x04, J5 Conn_01x04, J6 Conn_02x04_Odd_Even, U2 Value: Value: Value: Value: M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, U3 MCP2515-I/P, U4 TLP222A, U5 MAX31855, Y1 8MHz

Commit message: 更新
Connections:
- net +12V: no longer LS1.P, U4.4
- net +5V: now also LS1.P, U4.4
- net PhotoMos_12Vin: no longer names the net of R10.2, R11.2, U4.1
Changed lines of the file:
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@@
     (stroke (width 0) (type default))
   )
-  (wire (pts (xy 210.82 33.02) (xy 210.82 41.91))
+  (wire (pts (xy 210.82 39.37) (xy 210.82 41.91))
     (stroke (width 0) (type default))
   )
@@
   )
   (text "MAX31855 熱電対-デジタルコンバーター" (at 195.58 93.98 0)
-    (effects (font (size 1.27 1.27)) (justify left bottom))
-  )
-  (label "PhotoMos_12Vin" (at 194.31 41.91 90) (fields_autoplaced)
     (effects (font (size 1.27 1.27)) (justify left bottom))
   )
@@
     )
   )
-  (symbol (lib_id "power:+12V") (at 210.82 33.02 0) (unit 1)
-    (in_bom yes) (on_board yes) (dnp no) (fields_autoplaced)
-    (property "Reference" "#PWR042" (at 210.82 36.83 0)
-      (effects (font (size 1.27 1.27)) hide)
-    )
-    (property "Value" "+12V" (at 210.82 29.21 0)
-      (effects (font (size 1.27 1.27)))
-    )
-    (property "Footprint" "" (at 210.82 33.02 0)
-      (effects (font (size 1.27 1.27)) hide)
-    )
-    (property "Datasheet" "" (at 210.82 33.02 0)
-      (effects (font (size 1.27 1.27)) hide)
-    )
-    (pin "1")
-    (instances
-      (project "THRControlModuleBoard"
-        (path "/79fd2516-dad6-414c-bb46-91ee9bfb5006/c651c84e-0d0e-46aa-94b6-456d48525723"
-          (reference "#PWR042") (unit 1)
-        )
-      )
-    )
-  )
   (symbol (lib_id "Diode:MM3Zxx") (at 31.75 59.69 90) (unit 1)
     (in_bom yes) (on_board yes) (dnp no) (fields_autoplaced)
@@
         )
       )
+    )
+  )
+  (symbol (lib_id "power:+5V") (at 210.82 39.37 0) (unit 1)
+    (in_bom yes) (on_board yes) (dnp no) (fields_autoplaced)
+    (property "Reference" "#PWR042" (at 210.82 43.18 0)
+      (effects (font (size 1.27 1.27)) hide)
+    )
+    (property "Value" "+5V" (at 210.82 35.56 0)
+      (effects (font (size 1.27 1.27)))
+    )
+    (property "Footprint" "" (at 210.82 39.37 0)
+      (effects (font (size 1.27 1.27)) hide)
+    )
+    (property "Datasheet" "" (at 210.82 39.37 0)
+      (effects (font (size 1.27 1.27)) hide)
+    )
+    (pin "1")
+    (instances
+      (project "THRControlModuleBoard"
+        (path "/79fd2516-dad6-414c-bb46-91ee9bfb5006/c651c84e-0d0e-46aa-94b6-456d48525723"
+          (reference "#PWR042") (unit 1)
+        )
+      )

Commit message: 長時間の動作を確認した。
Parts:
- removed R10: 620, Resistor_SMD:R_0603_1608Metric_Pad0.98x0.95mm_HandSolder, symbol Device:R
- removed R11: 300, Resistor_SMD:R_0603_1608Metric_Pad0.98x0.95mm_HandSolder, symbol Device:R
- removed U4: TLP222A, Package_DIP:DIP-4_W7.62mm, symbol Relay_SolidState:TLP222A
Connections:
- net +5V: no longer LS1.P
- net IO__Busser: now also LS1.P
Other:
- moved on the sheet: LS1
