File: Projects/KiCad/SensingModule/SensingModule.kicad_pcb (KiCad board)
At the start: 2 copper layers, 110 x 95 mm, 42 parts, among them J1 Conn_01x02, J2 Conn_01x08, J3 Conn_01x02_Pin, J4 Micro_SD_Card_Det_Hirose_DM3AT, SW1 SW_Push, SW2 SW_Push, U1 MCP2562-E-P, U4 TLP222A, U5 NUCLEO-F303K8, U6 MB85RS2MT, U7 MB85RS2MT

Commit message: 裏面にQRコードと署名を追加
Parts:
- added G***: LOGO, LOGO, B.Cu at (148.0, 60.5)
- added G***: LOGO, LOGO, B.Cu at (146.5, 70.5)
- added REF**: Bosch_LGA-8_3x3mm_P0.8mm_ClockwisePinNumbering, Package_LGA:Bosch_LGA-8_3x3mm_P0.8mm_ClockwisePinNumbering, F.Cu at (172.5, 85.6)
- added REF**: LGA-28_5.2x3.8mm_P0.5mm, Package_LGA:LGA-28_5.2x3.8mm_P0.5mm, F.Cu at (172.4, 96.5)
Routing:
- net DUMP_MODE: track 53.9 -> 52.6 mm
Other:
- board text added: "Designed by Y.Iwai 2023"
- board text added: "Sensing Module Build 1"
- board text added: "Tokai Student Rocket Poject H-58 Avionics"
