File: Projects/KiCad/Structures/AvionicsMountPlate/AvionicsMountPlate.kicad_pcb (KiCad board)
At the start: 2 copper layers, 140 x 140 mm, 41 parts

Commit message: 許されざる基板を修正
Parts:
- removed the G*** at (176.3, 106.4)
- removed the G*** at (149.6, 87.4)
- removed the G*** at (178.8, 87.4)
- removed the G*** at (159.8, 116.6)
- removed the G*** at (121.7, 105.2)
- removed the G*** at (144.5, 105.2)
- removed the G*** at (126.8, 87.4)
- removed the G*** at (136.9, 116.6)
- moved G*** 6.35 mm to (149.6, 76.0)

Commit message: コネクタ位置を揃えた
Parts:
- removed the G*** at (149.6, 87.4)
