File: Projects/KiCad/Modules/CommunicationModule/AirData/AirData.kicad_pcb (KiCad board)
At the start: 2 copper layers, 110 x 95 mm, 36 parts, among them J1 Conn_01x08, SW1 SW_DIP_x02, U1 MCP2562-E-P, U2 MCP2515-I/P, U3 NJM7805SDL1, U4 ABX00012, Y1 8MHz

Commit message: チェックよし（多分）
Changed lines of the file:
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@@
     (fp_line (start 1 0.625) (end -1 0.625)
       (stroke (width 0.1) (type solid)) (layer "F.Fab"))
-    (pad "1" smd roundrect (at -1 0 270) (size 1.2 1.4) (layers "F.Cu" "F.Paste" "F.Mask") (roundrect_rratio 0.208333)
+    (pad "1" smd roundrect (at -1 0 270) (size 1.2 1.4) (layers "F.Cu" "F.Paste" "F.Mask") (roundrect_rratio 0.2083333333)
       (net 32 "CAN_RECEIVE_STATUS") (pintype "passive"))
-    (pad "2" smd roundrect (at 1 0 270) (size 1.2 1.4) (layers "F.Cu" "F.Paste" "F.Mask") (roundrect_rratio 0.208333)
+    (pad "2" smd roundrect (at 1 0 270) (size 1.2 1.4) (layers "F.Cu" "F.Paste" "F.Mask") (roundrect_rratio 0.2083333333)
       (net 29 "Net-(D3-A)") (pintype "passive"))
     (model "${KICAD6_3DMODEL_DIR}/Resistor_SMD.3dshapes/R_0805_2012Metric.wrl"
@@
     (fp_line (start 1 0.625) (end -1 0.625)
       (stroke (width 0.1) (type solid)) (layer "F.Fab"))
-    (pad "1" smd roundrect (at -1 0 270) (size 1.2 1.4) (layers "F.Cu" "F.Paste" "F.Mask") (roundrect_rratio 0.208333)
+    (pad "1" smd roundrect (at -1 0 270) (size 1.2 1.4) (layers "F.Cu" "F.Paste" "F.Mask") (roundrect_rratio 0.2083333333)
       (net 34 "LORA_RECEIVE_STATUS") (pintype "passive"))
-    (pad "2" smd roundrect (at 1 0 270) (size 1.2 1.4) (layers "F.Cu" "F.Paste" "F.Mask") (roundrect_rratio 0.208333)
+    (pad "2" smd roundrect (at 1 0 270) (size 1.2 1.4) (layers "F.Cu" "F.Paste" "F.Mask") (roundrect_rratio 0.2083333333)
       (net 31 "Net-(D5-A)") (pintype "passive"))
     (model "${KICAD6_3DMODEL_DIR}/Resistor_SMD.3dshapes/R_0805_2012Metric.wrl"
@@
     (fp_line (start 1 0.625) (end -1 0.625)
       (stroke (width 0.1) (type solid)) (layer "F.Fab"))
-    (pad "1" smd roundrect (at -1 0 270) (size 1.2 1.4) (layers "F.Cu" "F.Paste" "F.Mask") (roundrect_rratio 0.208333)
+    (pad "1" smd roundrect (at -1 0 270) (size 1.2 1.4) (layers "F.Cu" "F.Paste" "F.Mask") (roundrect_rratio 0.2083333333)
       (net 35 "LORA_SEND_STATUS") (pintype "passive"))
-    (pad "2" smd roundrect (at 1 0 270) (size 1.2 1.4) (layers "F.Cu" "F.Paste" "F.Mask") (roundrect_rratio 0.208333)
+    (pad "2" smd roundrect (at 1 0 270) (size 1.2 1.4) (layers "F.Cu" "F.Paste" "F.Mask") (roundrect_rratio 0.2083333333)
       (net 14 "Net-(D6-A)") (pintype "passive"))
     (model "${KICAD6_3DMODEL_DIR}/Resistor_SMD.3dshapes/R_0805_2012Metric.wrl"
@@
     (fp_line (start 1 0.625) (end -1 0.625)
       (stroke (width 0.1) (type solid)) (layer "F.Fab"))
-    (pad "1" smd roundrect (at -1 0 270) (size 1.2 1.4) (layers "F.Cu" "F.Paste" "F.Mask") (roundrect_rratio 0.208333)
+    (pad "1" smd roundrect (at -1 0 270) (size 1.2 1.4) (layers "F.Cu" "F.Paste" "F.Mask") (roundrect_rratio 0.2083333333)
       (net 33 "CAN_SEND_STATUS") (pintype "passive"))
-    (pad "2" smd roundrect (at 1 0 270) (size 1.2 1.4) (layers "F.Cu" "F.Paste" "F.Mask") (roundrect_rratio 0.208333)
+    (pad "2" smd roundrect (at 1 0 270) (size 1.2 1.4) (layers "F.Cu" "F.Paste" "F.Mask") (roundrect_rratio 0.2083333333)
       (net 28 "Net-(D2-A)") (pintype "passive"))
     (model "${KICAD6_3DMODEL_DIR}/Resistor_SMD.3dshapes/R_0805_2012Metric.wrl"
@@
     (fp_line (start 1 0.625) (end -1 0.625)
       (stroke (width 0.1) (type solid)) (layer "F.Fab"))
-    (pad "1" smd roundrect (at -1 0) (size 1.2 1.4) (layers "F.Cu" "F.Paste" "F.Mask") (roundrect_rratio 0.208333)
+    (pad "1" smd roundrect (at -1 0) (size 1.2 1.4) (layers "F.Cu" "F.Paste" "F.Mask") (roundrect_rratio 0.2083333333)
       (net 5 "+3.3V") (pintype "passive"))
-    (pad "2" smd roundrect (at 1 0) (size 1.2 1.4) (layers "F.Cu" "F.Paste" "F.Mask") (roundrect_rratio 0.208333)
+    (pad "2" smd roundrect (at 1 0) (size 1.2 1.4) (layers "F.Cu" "F.Paste" "F.Mask") (roundrect_rratio 0.2083333333)
       (net 15 "Net-(U2-~RESET)") (pintype "passive"))
     (model "${KICAD6_3DMODEL_DIR}/Resistor_SMD.3dshapes/R_0805_2012Metric.wrl"

Commit message: 配線の繋ぎ忘れを修正
Connections:
- U4 pad 25: unconnected-(U4-GND-Pad25) -> GND
Changed lines of the file:
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@@
   (net 45 "unconnected-(U4-PB22_S5_TX-Pad23)")
   (net 46 "unconnected-(U4-RESET-Pad24)")
-  (net 47 "unconnected-(U4-GND-Pad25)")
-  (net 48 "unconnected-(U4-+5V-Pad28)")
-  (net 49 "+12V")
-  (net 50 "unconnected-(SW1-Pad2)")
-  (net 51 "unconnected-(SW1-Pad3)")
+  (net 47 "unconnected-(U4-+5V-Pad28)")
+  (net 48 "+12V")
+  (net 49 "unconnected-(SW1-Pad2)")
+  (net 50 "unconnected-(SW1-Pad3)")
   (footprint "MountingHole:MountingHole_4.5mm" locked (layer "F.Cu")
     (at 178.5 75)
@@
       (stroke (width 0.1) (type solid)) (layer "F.Fab"))
     (pad "1" smd roundrect (at -0.8625 0 180) (size 1.075 0.95) (layers "F.Cu" "F.Paste" "F.Mask") (roundrect_rratio 0.25)
-      (net 49 "+12V") (pintype "passive"))
+      (net 48 "+12V") (pintype "passive"))
     (pad "2" smd roundrect (at 0.8625 0 180) (size 1.075 0.95) (layers "F.Cu" "F.Paste" "F.Mask") (roundrect_rratio 0.25)
       (net 2 "GND") (pintype "passive"))
@@
       (stroke (width 0.1) (type solid)) (fill solid) (layer "F.SilkS"))
     (pad "1" thru_hole roundrect (at 0 0) (size 1.2 1.62) (drill 0.85) (layers "*.Cu" "*.Mask") (roundrect_rratio 0.2083333333)
-      (net 49 "+12V") (pinfunction "Pin_1") (pintype "passive"))
+      (net 48 "+12V") (pinfunction "Pin_1") (pintype "passive"))
     (pad "2" thru_hole oval (at 0 2) (size 1.2 1.65) (drill 0.85) (layers "*.Cu" "*.Mask")
-      (net 49 "+12V") (pinfunction "Pin_2") (pintype "passive"))
+      (net 48 "+12V") (pinfunction "Pin_2") (pintype "passive"))
     (pad "3" thru_hole oval (at 2 0) (size 1.2 1.65) (drill 0.85) (layers "*.Cu" "*.Mask")
       (net 2 "GND") (pinfunction "Pin_3") (pintype "passive"))
@@
       (net 46 "unconnected-(U4-RESET-Pad24)") (pinfunction "RESET") (pintype "input+no_connect"))
     (pad "25" thru_hole circle locked (at 29.7548 -22.66 270) (size 1.508 1.508) (drill 1) (layers "*.Cu" "*.Mask")
-      (net 47 "unconnected-(U4-GND-Pad25)") (pinfunction "GND") (pintype "power_in+no_connect"))
+      (net 2 "GND") (pinfunction "GND") (pintype "power_in"))
     (pad "26" thru_hole circle locked (at 27.2148 -22.66 270) (size 1.508 1.508) (drill 1) (layers "*.Cu" "*.Mask")
       (net 5 "+3.3V") (pinfunction "+3V3") (pintype "power_in"))
@@
       (net 3 "+5V") (pinfunction "VIN") (pintype "power_in"))
     (pad "28" thru_hole circle locked (at 22.1348 -22.66 270) (size 1.508 1.508) (drill 1) (layers "*.Cu" "*.Mask")
-      (net 48 "unconnected-(U4-+5V-Pad28)") (pinfunction "+5V") (pintype "power_in+no_connect"))
+      (net 47 "unconnected-(U4-+5V-Pad28)") (pinfunction "+5V") (pintype "power_in+no_connect"))
     (model "/Users/waiwai/Projects/H-58-Avionics/Projects/KiCad/Modules/ReadyMadeModules/Arduino MKR WAN 1310/Arduino MKR WAN 1310.step"
       (offset (xyz 0 0 2.5))
@@
       (net 36 "DEBUG_MODE") (pintype "passive"))
     (pad "2" thru_hole oval (at 0 2.54 270) (size 1.6 1.6) (drill 0.8) (layers "*.Cu" "*.Mask")
-      (net 50 "unconnected-(SW1-Pad2)") (pintype "passive"))
+      (net 49 "unconnected-(SW1-Pad2)") (pintype "passive"))
     (pad "3" thru_hole oval (at 7.62 2.54 270) (size 1.6 1.6) (drill 0.8) (layers "*.Cu" "*.Mask")
-      (net 51 "unconnected-(SW1-Pad3)") (pintype "passive"))
+      (net 50 "unconnected-(SW1-Pad3)") (pintype "passive"))
     (pad "4" thru_hole oval (at 7.62 0 270) (size 1.6 1.6) (drill 0.8) (layers "*.Cu" "*.Mask")
       (net 2 "GND") (pintype "passive"))
@@
       (stroke (width 0.1) (type solid)) (layer "F.Fab"))
     (pad "1" smd roundrect (at -1.4 0 90) (size 1.1 1.1) (layers "F.Cu" "F.Paste" "F.Mask") (roundrect_rratio 0.2272727273)
-      (net 49 "+12V") (pinfunction "K") (pintype "passive"))
+      (net 48 "+12V") (pinfunction "K") (pintype "passive"))
     (pad "2" smd roundrect (at 1.4 0 90) (size 1.1 1.1) (layers "F.Cu" "F.Paste" "F.Mask") (roundrect_rratio 0.2272727273)
       (net 3 "+5V") (pinfunction "A") (pintype "passive"))
@@
       (stroke (width 0.1) (type solid)) (layer "F.Fab"))
     (pad "1" smd roundrect (at -5.04 -2.28 180) (size 2.2 1.2) (layers "F.Cu" "F.Paste" "F.Mask") (roundrect_rratio 0.2083333333)
-      (net 49 "+12V") (pinfunction "IN") (pintype "power_in"))
+      (net 48 "+12V") (pinfunction "IN") (pintype "power_in"))
     (pad "2" smd roundrect (at -0.415 -1.525 180) (size 3.05 2.75) (layers "F.Cu" "F.Paste") (roundrect_rratio 0.09090909091)
       (net 2 "GND") (pinfunction "GND") (pintype "power_in"))
@@
   (segment (start 133.475 59.874432) (end 134.4773 60.876732) (width 0.3) (layer "F.Cu") (net 36))
   (segment (start 136.86845 96.6798) (end 138.0798 96.6798) (width 0.3) (layer "F.Cu") (net 36))
-  (segment (start 161.9548 131.9548) (end 161.9548 129.1002) (width 1) (layer "F.Cu") (net 49))
-  (segment (start 162 132) (end 161.9548 131.9548) (width 1) (layer "F.Cu") (net 49))
-  (segment (start 162 132) (end 162 134) (width 1) (layer "F.Cu") (net 49))
-  (segment (start 174.32 114.179432) (end 175.2 113.299432) (width 1) (layer "F.Cu") (net 49))
-  (segment (start 172.3 114.179432) (end 174.32 114.179432) (width 1) (layer "F.Cu") (net 49))
-  (segment (start 171.8875 119.1675) (end 171.8875 116.949432) (width 1) (layer "F.Cu") (net 49))
-  (segment (start 161.9548 129.1002) (end 171.8875 119.1675) (width 1) (layer "F.Cu") (net 49))
-  (segment (start 171.8875 116.949432) (end 172.3 116.536932) (width 1) (layer "F.Cu") (net 49))
-  (segment (start 172.3 116.536932) (end 172.3 114.179432) (width 1) (layer "F.Cu") (net 49))
+  (segment (start 161.9548 131.9548) (end 161.9548 129.1002) (width 1) (layer "F.Cu") (net 48))
+  (segment (start 162 132) (end 161.9548 131.9548) (width 1) (layer "F.Cu") (net 48))
+  (segment (start 162 132) (end 162 134) (width 1) (layer "F.Cu") (net 48))
+  (segment (start 174.32 114.179432) (end 175.2 113.299432) (width 1) (layer "F.Cu") (net 48))
+  (segment (start 172.3 114.179432) (end 174.32 114.179432) (width 1) (layer "F.Cu") (net 48))
+  (segment (start 171.8875 119.1675) (end 171.8875 116.949432) (width 1) (layer "F.Cu") (net 48))
+  (segment (start 161.9548 129.1002) (end 171.8875 119.1675) (width 1) (layer "F.Cu") (net 48))
+  (segment (start 171.8875 116.949432) (end 172.3 116.536932) (width 1) (layer "F.Cu") (net 48))
+  (segment (start 172.3 116.536932) (end 172.3 114.179432) (width 1) (layer "F.Cu") (net 48))
   (zone (net 3) (net_name "+5V") (layer "F.Cu") (name "$teardrop_padvia$") (hatch edge 0.5)
     (priority 30066)
@@
     )
   )
-  (zone (net 49) (net_name "+12V") (layer "F.Cu") (name "$teardrop_padvia$") (hatch edge 0.5)
+  (zone (net 48) (net_name "+12V") (layer "F.Cu") (name "$teardrop_padvia$") (hatch edge 0.5)
     (priority 30029)
     (attr (teardrop (type padvia)))
@@
     )
   )
-  (zone (net 49) (net_name "+12V") (layer "F.Cu") (name "$teardrop_padvia$") (hatch edge 0.5)
+  (zone (net 48) (net_name "+12V") (layer "F.Cu") (name "$teardrop_padvia$") (hatch edge 0.5)
     (priority 30007)
     (attr (teardrop (type padvia)))
@@
     )
   )
-  (zone (net 49) (net_name "+12V") (layer "F.Cu") (name "$teardrop_padvia$") (hatch edge 0.5)
+  (zone (net 48) (net_name "+12V") (layer "F.Cu") (name "$teardrop_padvia$") (hatch edge 0.5)
     (priority 30008)
     (attr (teardrop (type padvia)))
@@
     )
   )
-  (zone (net 49) (net_name "+12V") (layer "F.Cu") (name "$teardrop_padvia$") (hatch edge 0.5)
+  (zone (net 48) (net_name "+12V") (layer "F.Cu") (name "$teardrop_padvia$") (hatch edge 0.5)
     (priority 30015)
     (attr (teardrop (type padvia)))
@@
     )
   )
-  (zone (net 49) (net_name "+12V") (layer "F.Cu") (name "$teardrop_padvia$") (hatch edge 0.5)
+  (zone (net 48) (net_name "+12V") (layer "F.Cu") (name "$teardrop_padvia$") (hatch edge 0.5)
     (priority 30016)
     (attr (teardrop (type padvia)))
