File: Projects/KiCad/Modules/CommunicationModule/AirData/AirData.kicad_pcb (KiCad board)
At the start: 2 copper layers, 110 x 95 mm, 36 parts, among them J1 Conn_01x08, SW1 SW_DIP_x02, U1 MCP2562-E-P, U2 MCP2515-I/P, U3 NJM7805SDL1, U4 ABX00012, Y1 8MHz

Commit message: ガーバーを再生成
Parts:
- C2: value 10μF -> 10uF
- C3, C4, C5, C6: value 0.1μF -> 0.1uF
- C8: value 47μF -> 47uF
- D2, D3, D5, D6: value ORANGE -> BLUE
- R1: value 120Ω -> 120R
- R2: value 620Ω -> 620R
- R3: value 10kΩ -> 10kR
- R4, R5, R6, R7: value 100Ω -> 100R
Changed lines of the file:
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@@
         (effects (font (size 1 1) (thickness 0.15)))
     )
-    (fp_text value "10μF" (at 0 1.43 180) (layer "F.Fab")
+    (fp_text value "10uF" (at 0 1.43 180) (layer "F.Fab")
         (effects (font (size 1 1) (thickness 0.15)))
     )
@@
         (effects (font (size 1 1) (thickness 0.15)))
     )
-    (fp_text value "0.1μF" (at 0 1.43 90) (layer "F.Fab")
+    (fp_text value "0.1uF" (at 0 1.43 90) (layer "F.Fab")
         (effects (font (size 1 1) (thickness 0.15)))
     )
@@
         (effects (font (size 1 1) (thickness 0.15)))
     )
-    (fp_text value "100Ω" (at 0 1.65 -90) (layer "F.Fab")
+    (fp_text value "100R" (at 0 1.65 -90) (layer "F.Fab")
         (effects (font (size 1 1) (thickness 0.15)))
     )
@@
         (effects (font (size 1 1) (thickness 0.15)))
     )
-    (fp_text value "0.1μF" (at 0 1.43 180) (layer "F.Fab")
+    (fp_text value "0.1uF" (at 0 1.43 180) (layer "F.Fab")
         (effects (font (size 1 1) (thickness 0.15)))
     )
@@
         (effects (font (size 1 1) (thickness 0.15)))
     )
-    (fp_text value "100Ω" (at 0 1.65 -90) (layer "F.Fab")
+    (fp_text value "100R" (at 0 1.65 -90) (layer "F.Fab")
         (effects (font (size 1 1) (thickness 0.15)))
     )
@@
         (effects (font (size 1 1) (thickness 0.15)))
     )
-    (fp_text value "100Ω" (at 0 1.65 -90) (layer "F.Fab")
+    (fp_text value "100R" (at 0 1.65 -90) (layer "F.Fab")
         (effects (font (size 1 1) (thickness 0.15)))
     )
@@
         (effects (font (size 1 1) (thickness 0.15)))
     )
-    (fp_text value "0.1μF" (at 0 1.43 90) (layer "F.Fab")
+    (fp_text value "0.1uF" (at 0 1.43 90) (layer "F.Fab")
         (effects (font (size 1 1) (thickness 0.15)))
     )
@@
         (effects (font (size 1 1) (thickness 0.15)))
     )
-    (fp_text value "0.1μF" (at 0 1.43 180) (layer "F.Fab")
+    (fp_text value "0.1uF" (at 0 1.43 180) (layer "F.Fab")
         (effects (font (size 1 1) (thickness 0.15)))
     )
@@
         (effects (font (size 1 1) (thickness 0.15)))
     )
-    (fp_text value "47μF" (at 0 4.35) (layer "F.Fab")
+    (fp_text value "47uF" (at 0 4.35) (layer "F.Fab")
         (effects (font (size 1 1) (thickness 0.15)))
     )
@@
         (effects (font (size 1 1) (thickness 0.15)))
     )
-    (fp_text value "ORANGE" (at 0 1.43 90) (layer "F.Fab")
+    (fp_text value "BLUE" (at 0 1.43 90) (layer "F.Fab")
         (effects (font (size 1 1) (thickness 0.15)))
     )
@@
         (effects (font (size 1 1) (thickness 0.15)))
     )
-    (fp_text value "100Ω" (at 0 1.65 -90) (layer "F.Fab")
+    (fp_text value "100R" (at 0 1.65 -90) (layer "F.Fab")
         (effects (font (size 1 1) (thickness 0.15)))
     )
@@
         (effects (font (size 1 1) (thickness 0.15)))
     )
-    (fp_text value "ORANGE" (at 0 1.43 90) (layer "F.Fab")
+    (fp_text value "BLUE" (at 0 1.43 90) (layer "F.Fab")
         (effects (font (size 1 1) (thickness 0.15)))
     )
@@
         (effects (font (size 1 1) (thickness 0.15)))
     )
-    (fp_text value "ORANGE" (at 0 1.43 90) (layer "F.Fab")
+    (fp_text value "BLUE" (at 0 1.43 90) (layer "F.Fab")
         (effects (font (size 1 1) (thickness 0.15)))
     )
@@
         (effects (font (size 1 1) (thickness 0.15)))
     )
-    (fp_text value "ORANGE" (at 0 1.43 90) (layer "F.Fab")
+    (fp_text value "BLUE" (at 0 1.43 90) (layer "F.Fab")
         (effects (font (size 1 1) (thickness 0.15)))
     )
@@
         (effects (font (size 1 1) (thickness 0.15)))
     )
-    (fp_text value "620Ω" (at 0 1.43) (layer "F.Fab")
+    (fp_text value "620R" (at 0 1.43) (layer "F.Fab")
         (effects (font (size 1 1) (thickness 0.15)))
     )
@@
         (effects (font (size 1 1) (thickness 0.15)))
     )
-    (fp_text value "120Ω" (at 0 1.43) (layer "F.Fab")
+    (fp_text value "120R" (at 0 1.43) (layer "F.Fab")
         (effects (font (size 1 1) (thickness 0.15)))
     )
@@
         (effects (font (size 1 1) (thickness 0.15)))
     )
-    (fp_text value "10kΩ" (at 0 1.65) (layer "F.Fab")
-        (effects (font (size 1 1) (thickness 0.15)))
-    )
+    (fp_text value "10kR" (at 0 1.65) (layer "F.Fab")
+        (effects (font (size 1 1) (thickness 0.15)))
+    )

Commit message: QRと署名を更新
Parts:
- moved G*** 0.71 mm to (148.5, 63.0), turned to 90 degrees
Other:
- board text added: "Communication Module Air Data Build 2"
- board text removed: "Communication Module Air Data Build 1"
