File: Projects/KiCad/Modules/MissionModule/MissionModule.kicad_sch (KiCad schematic)
At the start: 50 parts, among them J1 Conn_01x08, J2 Micro_SD_Card_Det_Hirose_DM3AT, SW1 SW_DIP_x02, U1 MCP2562-E-P, U2 MCP2515-I/P, U3 NJM7805SDL1, U5 TLP222A, U6 ABX00012, U7 MB85RS2MT, U8 MB85RS2MT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

Commit message: SPIのプルアップ電圧源をRECORDER_POWERに変更
Connections:
- net +3.3V: no longer R12.1, R13.1, R14.1
- net MEMORY_POWER: now also R12.1, R13.1, R14.1
Changed lines of the file:
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@@
+    (stroke (width 0) (type default))
+  )
+  (wire (pts (xy 99.06 121.92) (xy 101.6 121.92))
     (stroke (width 0) (type default))
   )
@@
     (stroke (width 0) (type default))
   )
+  (wire (pts (xy 36.83 121.92) (xy 36.83 124.46))
+    (stroke (width 0) (type default))
+  )
   (wire (pts (xy 152.4 177.8) (xy 152.4 184.15))
     (stroke (width 0) (type default))
@@
     (stroke (width 0) (type default))
   )
+  (wire (pts (xy 34.29 121.92) (xy 36.83 121.92))
+    (stroke (width 0) (type default))
+  )
   (wire (pts (xy 101.6 132.08) (xy 101.6 134.62))
     (stroke (width 0) (type default))
@@
     (stroke (width 0) (type default))
   )
-  (wire (pts (xy 36.83 121.92) (xy 36.83 124.46))
-    (stroke (width 0) (type default))
-  )
   (wire (pts (xy 44.45 121.92) (xy 57.15 121.92))
     (stroke (width 0) (type default))
@@
   )
   (wire (pts (xy 107.95 109.22) (xy 110.49 109.22))
+    (stroke (width 0) (type default))
+  )
+  (wire (pts (xy 158.75 113.03) (xy 161.29 113.03))
     (stroke (width 0) (type default))
   )
@@
     )
   )
+  (global_label "MEMORY_POWER" (shape input) (at 34.29 121.92 180) (fields_autoplaced)
+    (effects (font (size 1.27 1.27)) (justify right))
+    (property "Intersheetrefs" "${INTERSHEET_REFS}" (at 16.2048 121.92 0)
+      (effects (font (size 1.27 1.27)) (justify right) hide)
+    )
+  )
   (global_label "CAN_TX" (shape input) (at 107.95 44.45 0) (fields_autoplaced)
     (effects (font (size 1.27 1.27)) (justify left))
@@
     )
   )
+  (global_label "MEMORY_POWER" (shape input) (at 158.75 113.03 180) (fields_autoplaced)
+    (effects (font (size 1.27 1.27)) (justify right))
+    (property "Intersheetrefs" "${INTERSHEET_REFS}" (at 140.6648 113.03 0)
+      (effects (font (size 1.27 1.27)) (justify right) hide)
+    )
+  )
   (global_label "CAN_SEND_STATUS" (shape input) (at 232.41 40.64 90) (fields_autoplaced)
     (effects (font (size 1.27 1.27)) (justify left))
@@
     (effects (font (size 1.27 1.27)) (justify right))
     (property "Intersheetrefs" "${INTERSHEET_REFS}" (at 16.9681 55.88 0)
+      (effects (font (size 1.27 1.27)) (justify right) hide)
+    )
+  )
+  (global_label "MEMORY_POWER" (shape input) (at 99.06 121.92 180) (fields_autoplaced)
+    (effects (font (size 1.27 1.27)) (justify right))
+    (property "Intersheetrefs" "${INTERSHEET_REFS}" (at 80.9748 121.92 0)
       (effects (font (size 1.27 1.27)) (justify right) hide)
     )
@@
         (path "/ea1ed597-7cd3-4340-902e-bdce8f2d7a62"
           (reference "R9") (unit 1)
-        )
-      )
-    )
-  )
-  (symbol (lib_id "power:+3.3V") (at 36.83 121.92 0) (unit 1)
-    (in_bom yes) (on_board yes) (dnp no) (fields_autoplaced)
-    (property "Reference" "#PWR034" (at 36.83 125.73 0)
-      (effects (font (size 1.27 1.27)) hide)
-    )
-    (property "Value" "+3.3V" (at 36.83 118.11 0)
-      (effects (font (size 1.27 1.27)))
-    )
-    (property "Footprint" "" (at 36.83 121.92 0)
-      (effects (font (size 1.27 1.27)) hide)
-    )
-    (property "Datasheet" "" (at 36.83 121.92 0)
-      (effects (font (size 1.27 1.27)) hide)
-    )
-    (pin "1")
-    (instances
-      (project "MissionModule"
-        (path "/ea1ed597-7cd3-4340-902e-bdce8f2d7a62"
-          (reference "#PWR034") (unit 1)
         )
       )
@@
     )
   )
-  (symbol (lib_id "power:+3.3V") (at 101.6 121.92 0) (unit 1)
-    (in_bom yes) (on_board yes) (dnp no) (fields_autoplaced)
-    (property "Reference" "#PWR033" (at 101.6 125.73 0)
-      (effects (font (size 1.27 1.27)) hide)
-    )
-    (property "Value" "+3.3V" (at 101.6 118.11 0)
-      (effects (font (size 1.27 1.27)))
-    )
-    (property "Footprint" "" (at 101.6 121.92 0)
-      (effects (font (size 1.27 1.27)) hide)
-    )
-    (property "Datasheet" "" (at 101.6 121.92 0)
-      (effects (font (size 1.27 1.27)) hide)
-    )
-    (pin "1")
-    (instances
-      (project "MissionModule"
-        (path "/ea1ed597-7cd3-4340-902e-bdce8f2d7a62"
-          (reference "#PWR033") (unit 1)
-        )
-      )
-    )
-  )
   (symbol (lib_id "power:+12V") (at 52.07 50.8 0) (mirror y) (unit 1)
     (in_bom yes) (on_board yes) (dnp no) (fields_autoplaced)
@@
         )
       )
-    )
-  )
-  (symbol (lib_id "power:+3.3V") (at 161.29 113.03 0) (mirror y) (unit 1)
-    (in_bom yes) (on_board yes) (dnp no) (fields_autoplaced)
-    (property "Reference" "#PWR027" (at 161.29 116.84 0)
-      (effects (font (size 1.27 1.27)) hide)
-    )
-    (property "Value" "+3.3V" (at 161.29 109.22 0)
-      (effects (font (size 1.27 1.27)))
-    )
-    (property "Footprint" "" (at 161.29 113.03 0)
-      (effects (font (size 1.27 1.27)) hide)
-    )
-    (property "Datasheet" "" (at 161.29 113.03 0)
-      (effects (font (size 1.27 1.27)) hide)
-    )
-    (pin "1")
-    (instances
-      (project "MissionModule"
-        (path "/ea1ed597-7cd3-4340-902e-bdce8f2d7a62"
-          (reference "#PWR027") (unit 1)
-        )
-      )

Commit message: ガーバーを再生成
Parts:
- C2, C4, C5, C7: value 0.1μF -> 0.1uF
- C3: value 10μF -> 10uF
- C8, C9: value 47μF -> 47uF
- D3, D4, D5, D6: value ORANGE -> BLUE
- R1, R10, R8: value 120Ω -> 120R
- R11, R15, R9: value 300Ω -> 300R
- R12, R13, R14, R16: value 4.7kΩ -> 4.7kR
- R2: value 620Ω -> 620R
- R3: value 10kΩ -> 10kR
- R4, R5, R6, R7: value 100Ω -> 100R
- U4: value ~ -> ADXL375
- U5: value TLP222A -> TLP241B
Changed lines of the file:
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@@
       (effects (font (size 1.27 1.27)) (justify left))
     )
-    (property "Value" "620Ω" (at 215.9 48.2599 0)
+    (property "Value" "620R" (at 215.9 48.2599 0)
       (effects (font (size 1.27 1.27)) (justify left))
     )
@@
       (effects (font (size 1.27 1.27)) (justify left))
     )
-    (property "Value" "0.1μF" (at 252.73 111.125 0)
+    (property "Value" "0.1uF" (at 252.73 111.125 0)
       (effects (font (size 1.27 1.27)) (justify left))
     )
@@
       (effects (font (size 1.27 1.27)) (justify left))
     )
-    (property "Value" "100Ω" (at 274.32 48.2599 0)
+    (property "Value" "100R" (at 274.32 48.2599 0)
       (effects (font (size 1.27 1.27)) (justify left))
     )
@@
       (effects (font (size 1.27 1.27)))
     )
-    (property "Value" "10kΩ" (at 133.35 63.5 90)
+    (property "Value" "10kR" (at 133.35 63.5 90)
       (effects (font (size 1.27 1.27)))
     )
@@
       (effects (font (size 1.27 1.27)) (justify left))
     )
-    (property "Value" "300Ω" (at 255.27 48.2599 0)
+    (property "Value" "300R" (at 255.27 48.2599 0)
       (effects (font (size 1.27 1.27)) (justify left))
     )
@@
       (effects (font (size 1.27 1.27)) (justify right))
     )
-    (property "Value" "ORANGE" (at 236.22 60.0074 90)
+    (property "Value" "BLUE" (at 236.22 60.0074 90)
       (effects (font (size 1.27 1.27)) (justify right))
     )
@@
       (effects (font (size 1.27 1.27)) (justify left))
     )
-    (property "Value" "0.1μF" (at 86.36 29.21 0)
+    (property "Value" "0.1uF" (at 86.36 29.21 0)
       (effects (font (size 1.27 1.27)) (justify left))
     )
@@
       (effects (font (size 1.27 1.27)) (justify left))
     )
-    (property "Value" "4.7kΩ" (at 102.87 129.54 0)
+    (property "Value" "4.7kR" (at 102.87 129.54 0)
       (effects (font (size 1.27 1.27)) (justify left))
     )
@@
       (effects (font (size 1.27 1.27)) (justify left))
     )
-    (property "Value" "4.7kΩ" (at 38.1 129.54 0)
+    (property "Value" "4.7kR" (at 38.1 129.54 0)
       (effects (font (size 1.27 1.27)) (justify left))
     )
@@
       (effects (font (size 1.27 1.27)) (justify left))
     )
-    (property "Value" "10μF" (at 227.33 111.125 0)
+    (property "Value" "10uF" (at 227.33 111.125 0)
       (effects (font (size 1.27 1.27)) (justify left))
     )
@@
       (effects (font (size 1.27 1.27)) (justify left))
     )
-    (property "Value" "120Ω" (at 160.02 180.975 0)
+    (property "Value" "120R" (at 160.02 180.975 0)
       (effects (font (size 1.27 1.27)) (justify left))
     )
@@
       (effects (font (size 1.27 1.27)) (justify left))
     )
-    (property "Value" "0.1μF" (at 129.54 25.4 0)
+    (property "Value" "0.1uF" (at 129.54 25.4 0)
       (effects (font (size 1.27 1.27)) (justify left))
     )
@@
       (effects (font (size 1.27 1.27)) (justify right))
     )
-    (property "Value" "ORANGE" (at 285.75 60.0074 90)
+    (property "Value" "BLUE" (at 285.75 60.0074 90)
       (effects (font (size 1.27 1.27)) (justify right))
     )
@@
       (effects (font (size 1.27 1.27)) (justify left))
     )
-    (property "Value" "4.7kΩ" (at 160.02 120.65 0)
+    (property "Value" "4.7kR" (at 160.02 120.65 0)
       (effects (font (size 1.27 1.27)) (justify left))
     )
@@
       (effects (font (size 1.27 1.27)))
     )
-    (property "Value" "~" (at 63.5 168.91 0)
+    (property "Value" "ADXL375" (at 63.5 168.91 0)
       (effects (font (size 1.27 1.27)))
     )
@@
       (effects (font (size 1.27 1.27)) (justify left))
     )
-    (property "Value" "0.1μF" (at 77.47 29.21 0)
+    (property "Value" "0.1uF" (at 77.47 29.21 0)
       (effects (font (size 1.27 1.27)) (justify left))
     )
@@
       (effects (font (size 1.27 1.27)) (justify left))
     )
-    (property "Value" "300Ω" (at 265.43 48.2599 0)
+    (property "Value" "300R" (at 265.43 48.2599 0)
       (effects (font (size 1.27 1.27)) (justify left))
     )
@@
       (effects (font (size 1.27 1.27)) (justify left))
     )
-    (property "Value" "120Ω" (at 160.02 168.275 0)
+    (property "Value" "120R" (at 160.02 168.275 0)
       (effects (font (size 1.27 1.27)) (justify left))
     )
@@
       (effects (font (size 1.27 1.27)) (justify right))
     )
-    (property "Value" "ORANGE" (at 275.59 60.0074 90)
+    (property "Value" "BLUE" (at 275.59 60.0074 90)
       (effects (font (size 1.27 1.27)) (justify right))
     )
@@
       (effects (font (size 1.27 1.27)) (justify left))
     )
-    (property "Value" "47μF" (at 265.43 110.236 0)
+    (property "Value" "47uF" (at 265.43 110.236 0)
       (effects (font (size 1.27 1.27)) (justify left))
     )
@@
       (effects (font (size 1.27 1.27)) (justify left))
     )
-    (property "Value" "47μF" (at 123.19 185.166 0)
+    (property "Value" "47uF" (at 123.19 185.166 0)
       (effects (font (size 1.27 1.27)) (justify left))
     )
@@
       (effects (font (size 1.27 1.27)) (justify left))
     )
-    (property "Value" "100Ω" (at 284.48 48.2599 0)
+    (property "Value" "100R" (at 284.48 48.2599 0)
       (effects (font (size 1.27 1.27)) (justify left))
     )
@@
       (effects (font (size 1.27 1.27)) (justify left))
     )
-    (property "Value" "100Ω" (at 234.95 48.2599 0)
+    (property "Value" "100R" (at 234.95 48.2599 0)
       (effects (font (size 1.27 1.27)) (justify left))
     )
@@
       (effects (font (size 1.27 1.27)))
     )
-    (property "Value" "TLP222A" (at 142.24 180.34 0)
+    (property "Value" "TLP241B" (at 142.24 180.34 0)
       (effects (font (size 1.27 1.27)))
     )
@@
       (effects (font (size 1.27 1.27)) (justify left))
     )
-    (property "Value" "4.7kΩ" (at 34.29 175.26 0)
+    (property "Value" "4.7kR" (at 34.29 175.26 0)
       (effects (font (size 1.27 1.27)) (justify left))
     )
@@
       (effects (font (size 1.27 1.27)) (justify left))
     )
-    (property "Value" "120Ω" (at 72.39 50.8 0)
+    (property "Value" "120R" (at 72.39 50.8 0)
       (effects (font (size 1.27 1.27)) (justify left))
     )
@@
       (effects (font (size 1.27 1.27)) (justify left))
     )
-    (property "Value" "300Ω" (at 245.11 48.2599 0)
+    (property "Value" "300R" (at 245.11 48.2599 0)
       (effects (font (size 1.27 1.27)) (justify left))
     )
@@
       (effects (font (size 1.27 1.27)) (justify left))
     )
-    (property "Value" "100Ω" (at 224.79 48.2599 0)
+    (property "Value" "100R" (at 224.79 48.2599 0)
       (effects (font (size 1.27 1.27)) (justify left))
     )
@@
       (effects (font (size 1.27 1.27)) (justify right))
     )
-    (property "Value" "ORANGE" (at 226.06 60.0074 90)
+    (property "Value" "BLUE" (at 226.06 60.0074 90)
       (effects (font (size 1.27 1.27)) (justify right))
     )
