File: Projects/KiCad/Modules/MissionModule/MissionModule.kicad_pcb (KiCad board)
At the start: 2 copper layers, 110 x 95 mm, 56 parts, among them J1 Conn_01x08, J2 Micro_SD_Card_Det_Hirose_DM3AT, SW1 SW_DIP_x02, U1 MCP2562-E-P, U2 MCP2515-I/P, U3 NJM7805SDL1, U5 TLP222A, U6 ABX00012, U7 MB85RS2MT, U8 MB85RS2MT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

Commit message: 配線の繋ぎ忘れを修正
Connections:
- U6 pad 25: unconnected-(U6-GND-Pad25) -> GND

Commit message: FRAMのWPとHOLDをHIGHに固定
Connections:
- U7 pad 3: GND -> MEMORY_POWER
- U7 pad 7: GND -> MEMORY_POWER
- U8 pad 3: GND -> MEMORY_POWER
- U8 pad 7: GND -> MEMORY_POWER
Routing:
- net MEMORY_POWER: track 49.2 -> 78.6 mm

Commit message: SPIのプルアップ電圧源をRECORDER_POWERに変更
Connections:
- R12 pad 1: +3.3V -> MEMORY_POWER
- R13 pad 1: +3.3V -> MEMORY_POWER
- R14 pad 1: +3.3V -> MEMORY_POWER
Routing:
- net +3.3V: track 165.3 -> 144.4 mm
- net MEMORY_POWER: track 78.6 -> 89.0 mm

Commit message: ガーバーを再生成
Parts:
- C2, C4, C5, C7: value 0.1μF -> 0.1uF
- C3: value 10μF -> 10uF
- C8, C9: value 47μF -> 47uF
- D3, D4, D5, D6: value ORANGE -> BLUE
- R1, R10, R8: value 120Ω -> 120R
- R11, R15, R9: value 300Ω -> 300R
- R12, R13, R14, R16: value 4.7kΩ -> 4.7kR
- R2: value 620Ω -> 620R
- R3: value 10kΩ -> 10kR
- R4, R5, R6, R7: value 100Ω -> 100R
- U4: value ~ -> ADXL375
- U5: value TLP222A -> TLP241B
Changed lines of the file:
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@@
         (effects (font (size 1 1) (thickness 0.15)))
     )
-    (fp_text value "300Ω" (at 0 1.43) (layer "F.Fab")
+    (fp_text value "300R" (at 0 1.43) (layer "F.Fab")
         (effects (font (size 1 1) (thickness 0.15)))
     )
@@
         (effects (font (size 1 1) (thickness 0.15)))
     )
-    (fp_text value "4.7kΩ" (at 0 1.43) (layer "F.Fab")
+    (fp_text value "4.7kR" (at 0 1.43) (layer "F.Fab")
         (effects (font (size 1 1) (thickness 0.15)))
     )
@@
         (effects (font (size 1 1) (thickness 0.15)))
     )
-    (fp_text value "100Ω" (at 0 1.65 -90) (layer "F.Fab")
+    (fp_text value "100R" (at 0 1.65 -90) (layer "F.Fab")
         (effects (font (size 1 1) (thickness 0.15)))
     )
@@
         (effects (font (size 1 1) (thickness 0.15)))
     )
-    (fp_text value "0.1μF" (at 0 1.43 90) (layer "F.Fab")
+    (fp_text value "0.1uF" (at 0 1.43 90) (layer "F.Fab")
         (effects (font (size 1 1) (thickness 0.15)))
     )
@@
         (effects (font (size 1 1) (thickness 0.15)))
     )
-    (fp_text value "4.7kΩ" (at 0 1.43 90) (layer "F.Fab")
+    (fp_text value "4.7kR" (at 0 1.43 90) (layer "F.Fab")
         (effects (font (size 1 1) (thickness 0.15)))
     )
@@
         (effects (font (size 1 1) (thickness 0.15)))
     )
-    (fp_text value "10kΩ" (at 0 1.65) (layer "F.Fab")
+    (fp_text value "10kR" (at 0 1.65) (layer "F.Fab")
         (effects (font (size 1 1) (thickness 0.15)))
     )
@@
         (effects (font (size 1 1) (thickness 0.15)))
     )
-    (fp_text value "ORANGE" (at 0 1.43 90) (layer "F.Fab")
+    (fp_text value "BLUE" (at 0 1.43 90) (layer "F.Fab")
         (effects (font (size 1 1) (thickness 0.15)))
     )
@@
         (effects (font (size 1 1) (thickness 0.15)))
     )
-    (fp_text value "ORANGE" (at 0 1.43 90) (layer "F.Fab")
+    (fp_text value "BLUE" (at 0 1.43 90) (layer "F.Fab")
         (effects (font (size 1 1) (thickness 0.15)))
     )
@@
         (effects (font (size 1 1) (thickness 0.15)))
     )
-    (fp_text value "TLP222A" (at 3.81 4.87 90) (layer "F.Fab")
+    (fp_text value "TLP241B" (at 3.81 4.87 90) (layer "F.Fab")
         (effects (font (size 1 1) (thickness 0.15)))
     )
@@
         (effects (font (size 1 1) (thickness 0.15)))
     )
-    (fp_text value "300Ω" (at 0 1.43) (layer "F.Fab")
+    (fp_text value "300R" (at 0 1.43) (layer "F.Fab")
         (effects (font (size 1 1) (thickness 0.15)))
     )
@@
         (effects (font (size 1 1) (thickness 0.15)))
     )
-    (fp_text value "47μF" (at 0 4.35) (layer "F.Fab")
+    (fp_text value "47uF" (at 0 4.35) (layer "F.Fab")
         (effects (font (size 1 1) (thickness 0.15)))
     )
@@
         (effects (font (size 1 1) (thickness 0.15)))
     )
-    (fp_text value "100Ω" (at 0 1.65 -90) (layer "F.Fab")
+    (fp_text value "100R" (at 0 1.65 -90) (layer "F.Fab")
         (effects (font (size 1 1) (thickness 0.15)))
     )
@@
         (effects (font (size 1 1) (thickness 0.15)))
     )
-    (fp_text value "120Ω" (at 0 1.43 -90) (layer "F.Fab")
+    (fp_text value "120R" (at 0 1.43 -90) (layer "F.Fab")
         (effects (font (size 1 1) (thickness 0.15)))
     )
@@
         (effects (font (size 1 1) (thickness 0.15)))
     )
-    (fp_text value "100Ω" (at 0 1.65 -90) (layer "F.Fab")
+    (fp_text value "100R" (at 0 1.65 -90) (layer "F.Fab")
         (effects (font (size 1 1) (thickness 0.15)))
     )
@@
         (effects (font (size 1 1) (thickness 0.15)))
     )
-    (fp_text value "ORANGE" (at 0 1.43 90) (layer "F.Fab")
+    (fp_text value "BLUE" (at 0 1.43 90) (layer "F.Fab")
         (effects (font (size 1 1) (thickness 0.15)))
     )
@@
         (effects (font (size 1 1) (thickness 0.15)))
     )
-    (fp_text value "4.7kΩ" (at 0 1.43 90) (layer "F.Fab")
+    (fp_text value "4.7kR" (at 0 1.43 90) (layer "F.Fab")
         (effects (font (size 1 1) (thickness 0.15)))
     )
@@
         (effects (font (size 1 1) (thickness 0.15)))
     )
-    (fp_text value "ORANGE" (at 0 1.43 90) (layer "F.Fab")
+    (fp_text value "BLUE" (at 0 1.43 90) (layer "F.Fab")
         (effects (font (size 1 1) (thickness 0.15)))
     )
@@
         (effects (font (size 1 1) (thickness 0.15)))
     )
-    (fp_text value "~" (at 0 13.97 unlocked) (layer "F.Fab")
+    (fp_text value "ADXL375" (at 0 13.97 unlocked) (layer "F.Fab")
         (effects (font (size 1 1) (thickness 0.15)))
     )
@@
         (effects (font (size 1 1) (thickness 0.15)))
     )
-    (fp_text value "4.7kΩ" (at 0 1.43 90) (layer "F.Fab")
+    (fp_text value "4.7kR" (at 0 1.43 90) (layer "F.Fab")
         (effects (font (size 1 1) (thickness 0.15)))
     )
@@
         (effects (font (size 1 1) (thickness 0.15)))
     )
-    (fp_text value "0.1μF" (at 0 1.43 180) (layer "F.Fab")
+    (fp_text value "0.1uF" (at 0 1.43 180) (layer "F.Fab")
         (effects (font (size 1 1) (thickness 0.15)))
     )
@@
         (effects (font (size 1 1) (thickness 0.15)))
     )
-    (fp_text value "10μF" (at 0 1.43 180) (layer "F.Fab")
+    (fp_text value "10uF" (at 0 1.43 180) (layer "F.Fab")
         (effects (font (size 1 1) (thickness 0.15)))
     )
@@
         (effects (font (size 1 1) (thickness 0.15)))
     )
-    (fp_text value "47μF" (at 0 4.35 -90) (layer "F.Fab")
+    (fp_text value "47uF" (at 0 4.35 -90) (layer "F.Fab")
         (effects (font (size 1 1) (thickness 0.15)))
     )
@@
         (effects (font (size 1 1) (thickness 0.15)))
     )
-    (fp_text value "620Ω" (at 0 1.43) (layer "F.Fab")
+    (fp_text value "620R" (at 0 1.43) (layer "F.Fab")
         (effects (font (size 1 1) (thickness 0.15)))
     )
@@
         (effects (font (size 1 1) (thickness 0.15)))
     )
-    (fp_text value "0.1μF" (at 0 1.43 90) (layer "F.Fab")
+    (fp_text value "0.1uF" (at 0 1.43 90) (layer "F.Fab")
         (effects (font (size 1 1) (thickness 0.15)))
     )
@@
         (effects (font (size 1 1) (thickness 0.15)))
     )
-    (fp_text value "120Ω" (at 0 1.43) (layer "F.Fab")
+    (fp_text value "120R" (at 0 1.43) (layer "F.Fab")
         (effects (font (size 1 1) (thickness 0.15)))
     )
@@
         (effects (font (size 1 1) (thickness 0.15)))
     )
-    (fp_text value "120Ω" (at 0 1.43 -90) (layer "F.Fab")
+    (fp_text value "120R" (at 0 1.43 -90) (layer "F.Fab")
         (effects (font (size 1 1) (thickness 0.15)))
     )
@@
         (effects (font (size 1 1) (thickness 0.15)))
     )
-    (fp_text value "0.1μF" (at 0 1.43 180) (layer "F.Fab")
+    (fp_text value "0.1uF" (at 0 1.43 180) (layer "F.Fab")
         (effects (font (size 1 1) (thickness 0.15)))
     )
@@
         (effects (font (size 1 1) (thickness 0.15)))
     )
-    (fp_text value "100Ω" (at 0 1.65 -90) (layer "F.Fab")
+    (fp_text value "100R" (at 0 1.65 -90) (layer "F.Fab")
         (effects (font (size 1 1) (thickness 0.15)))
     )
@@
         (effects (font (size 1 1) (thickness 0.15)))
     )
-    (fp_text value "300Ω" (at 0 1.43 90) (layer "F.Fab")
-        (effects (font (size 1 1) (thickness 0.15)))
-    )
+    (fp_text value "300R" (at 0 1.43 90) (layer "F.Fab")
+        (effects (font (size 1 1) (thickness 0.15)))
+    )

Commit message: QRと署名を更新
Parts:
- moved G*** 1.22 mm to (148.2, 61.8)
Other:
- board text added: "Mission Module Build 2"
- board text removed: "Mission Module Build 1"
