File: Projects/KiCad/Modules/SensingModule/Recorder.kicad_sch (KiCad schematic)
At the start: 12 parts

Commit message: ガーバーを再生成
Parts:
- C?: value 47μF -> 47uF
- R? (x3): value 4.7kΩ -> 4.7kR
- R? (x2): value 120Ω -> 120R
- U?: value TLP222A -> TLP241B
Changed lines of the file:
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@@
       (effects (font (size 1.27 1.27)) (justify left))
     )
-    (property "Value" "4.7kΩ" (at 130.81 127 0)
+    (property "Value" "4.7kR" (at 130.81 127 0)
       (effects (font (size 1.27 1.27)) (justify left))
     )
@@
       (effects (font (size 1.27 1.27)) (justify left))
     )
-    (property "Value" "4.7kΩ" (at 48.26 127 0)
+    (property "Value" "4.7kR" (at 48.26 127 0)
       (effects (font (size 1.27 1.27)) (justify left))
     )
@@
       (effects (font (size 1.27 1.27)) (justify left))
     )
-    (property "Value" "120Ω" (at 85.09 66.675 0)
+    (property "Value" "120R" (at 85.09 66.675 0)
       (effects (font (size 1.27 1.27)) (justify left))
     )
@@
       (effects (font (size 1.27 1.27)) (justify left))
     )
-    (property "Value" "4.7kΩ" (at 210.82 113.03 0)
+    (property "Value" "4.7kR" (at 210.82 113.03 0)
       (effects (font (size 1.27 1.27)) (justify left))
     )
@@
       (effects (font (size 1.27 1.27)))
     )
-    (property "Value" "TLP222A" (at 67.31 66.04 0)
+    (property "Value" "TLP241B" (at 67.31 66.04 0)
       (effects (font (size 1.27 1.27)))
     )
@@
       (effects (font (size 1.27 1.27)) (justify left))
     )
-    (property "Value" "47μF" (at 48.26 70.866 0)
+    (property "Value" "47uF" (at 48.26 70.866 0)
       (effects (font (size 1.27 1.27)) (justify left))
     )
@@
       (effects (font (size 1.27 1.27)) (justify left))
     )
-    (property "Value" "120Ω" (at 85.09 53.975 0)
-      (effects (font (size 1.27 1.27)) (justify left))
-    )
+    (property "Value" "120R" (at 85.09 53.975 0)
+      (effects (font (size 1.27 1.27)) (justify left))
+    )
