File: Projects/KiCad/Modules/SensingModule/Sensor.kicad_sch (KiCad schematic)
At the start: 4 parts, among them J2 Conn_01x02_Pin

Commit message: ガーバーを再生成
Parts:
- R9: value 10kΩ -> 10kR
- U2: value ~ -> BME280
- U3: value ~ -> BNO055
Changed lines of the file:
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@@
       (effects (font (size 1.27 1.27)) (justify left))
     )
-    (property "Value" "~" (at 196.85 48.26 0)
+    (property "Value" "BME280" (at 196.85 48.26 0)
       (effects (font (size 1.27 1.27)))
     )
@@
       (effects (font (size 1.27 1.27)) (justify left))
     )
-    (property "Value" "10kΩ" (at 74.93 55.245 0)
+    (property "Value" "10kR" (at 74.93 55.245 0)
       (effects (font (size 1.27 1.27)) (justify left))
     )
@@
       (effects (font (size 1.27 1.27)) (justify left))
     )
-    (property "Value" "~" (at 137.16 57.15 0)
+    (property "Value" "BNO055" (at 137.16 57.15 0)
       (effects (font (size 1.27 1.27)))
     )
