File: Projects/KiCad/Modules/SensingModule/SensingModule.kicad_pcb (KiCad board)
At the start: 2 copper layers, 110 x 95 mm, 45 parts, among them J1 Conn_01x08, J2 Conn_01x02_Pin, J4 Micro_SD_Card_Det_Hirose_DM3AT, SW1 SW_DIP_x02, U1 MCP2562-E-P, U4 TLP222A, U5 NUCLEO-F303K8, U6 MB85RS2MT, U7 MB85RS2MT

Commit message: ガーバーを再生成
Parts:
- C1, C2: value 0.1μF -> 0.1uF
- C3: value 47μF -> 47uF
- D1, D2: value ORANGE -> BLUE
- R1, R3: value 100Ω -> 100R
- R10, R11, R15: value 300Ω -> 300R
- R12, R13, R14: value 4.7kΩ -> 4.7kR
- R2: value 120R1/4W -> 120R
- R4, R5, R9: value 10kΩ -> 10kR
- R6, R8: value 120Ω -> 120R
- R7: value 2kΩ -> 2kR
- U2: value ~ -> BME280
- U3: value ~ -> BNO055
- U4: value TLP222A -> TLP241B
Changed lines of the file:
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@@
         (effects (font (size 1 1) (thickness 0.15)))
     )
-    (fp_text value "100Ω" (at 0 1.65) (layer "F.Fab")
+    (fp_text value "100R" (at 0 1.65) (layer "F.Fab")
         (effects (font (size 1 1) (thickness 0.15)))
     )
@@
         (effects (font (size 1 1) (thickness 0.153)))
     )
-    (fp_text value "4.7kΩ" (at 0 1.43 90) (layer "F.Fab")
+    (fp_text value "4.7kR" (at 0 1.43 90) (layer "F.Fab")
         (effects (font (size 1 1) (thickness 0.15)))
     )
@@
         (effects (font (size 1 1) (thickness 0.153)))
     )
-    (fp_text value "~" (at 7.62 -2.77 180 unlocked) (layer "F.Fab")
+    (fp_text value "BME280" (at 7.62 -2.77 180 unlocked) (layer "F.Fab")
         (effects (font (size 1 1) (thickness 0.15)))
     )
@@
         (effects (font (size 1 1) (thickness 0.153)))
     )
-    (fp_text value "2kΩ" (at 0 1.43) (layer "F.Fab")
+    (fp_text value "2kR" (at 0 1.43) (layer "F.Fab")
         (effects (font (size 1 1) (thickness 0.15)))
     )
@@
         (effects (font (size 1 1) (thickness 0.153)))
     )
-    (fp_text value "4.7kΩ" (at 0 1.43 90) (layer "F.Fab")
+    (fp_text value "4.7kR" (at 0 1.43 90) (layer "F.Fab")
         (effects (font (size 1 1) (thickness 0.15)))
     )
@@
         (effects (font (size 1 1) (thickness 0.153)))
     )
-    (fp_text value "300Ω" (at 0 1.43) (layer "F.Fab")
+    (fp_text value "300R" (at 0 1.43) (layer "F.Fab")
         (effects (font (size 1 1) (thickness 0.15)))
     )
@@
         (effects (font (size 1 1) (thickness 0.153)))
     )
-    (fp_text value "300Ω" (at 0 1.43) (layer "F.Fab")
+    (fp_text value "300R" (at 0 1.43) (layer "F.Fab")
         (effects (font (size 1 1) (thickness 0.15)))
     )
@@
         (effects (font (size 1 1) (thickness 0.15)))
     )
-    (fp_text value "0.1μF" (at 0 1.43 90) (layer "F.Fab")
+    (fp_text value "0.1uF" (at 0 1.43 90) (layer "F.Fab")
         (effects (font (size 1 1) (thickness 0.15)))
     )
@@
         (effects (font (size 1 1) (thickness 0.153)))
     )
-    (fp_text value "ORANGE" (at 0 1.43) (layer "F.Fab")
+    (fp_text value "BLUE" (at 0 1.43) (layer "F.Fab")
         (effects (font (size 1 1) (thickness 0.15)))
     )
@@
         (effects (font (size 1 1) (thickness 0.15)))
     )
-    (fp_text value "100Ω" (at 0 1.65) (layer "F.Fab")
+    (fp_text value "100R" (at 0 1.65) (layer "F.Fab")
         (effects (font (size 1 1) (thickness 0.15)))
     )
@@
         (effects (font (size 1 1) (thickness 0.153)))
     )
-    (fp_text value "120Ω" (at 0 1.43 -90) (layer "F.Fab")
+    (fp_text value "120R" (at 0 1.43 -90) (layer "F.Fab")
         (effects (font (size 1 1) (thickness 0.15)))
     )
@@
         (effects (font (size 1 1) (thickness 0.153)))
     )
-    (fp_text value "TLP222A" (at 3.81 4.87 90) (layer "F.Fab")
+    (fp_text value "TLP241B" (at 3.81 4.87 90) (layer "F.Fab")
         (effects (font (size 1 1) (thickness 0.15)))
     )
@@
         (effects (font (size 1 1) (thickness 0.153)))
     )
-    (fp_text value "ORANGE" (at 0 1.43) (layer "F.Fab")
+    (fp_text value "BLUE" (at 0 1.43) (layer "F.Fab")
         (effects (font (size 1 1) (thickness 0.15)))
     )
@@
         (effects (font (size 1 1) (thickness 0.153)))
     )
-    (fp_text value "120R1/4W" (at 0 3.0175 90) (layer "F.Fab")
+    (fp_text value "120R" (at 0 3.0175 90) (layer "F.Fab")
         (effects (font (size 1 1) (thickness 0.15)))
     )
@@
         (effects (font (size 1 1) (thickness 0.15)))
     )
-    (fp_text value "10kΩ" (at 0 1.65 90) (layer "F.Fab")
+    (fp_text value "10kR" (at 0 1.65 90) (layer "F.Fab")
         (effects (font (size 1 1) (thickness 0.15)))
     )
@@
         (effects (font (size 1 1) (thickness 0.15)))
     )
-    (fp_text value "10kΩ" (at 0 1.65 90) (layer "F.Fab")
+    (fp_text value "10kR" (at 0 1.65 90) (layer "F.Fab")
         (effects (font (size 1 1) (thickness 0.15)))
     )
@@
         (effects (font (size 1 1) (thickness 0.153)))
     )
-    (fp_text value "~" (at 0 19.05 -90 unlocked) (layer "F.Fab")
+    (fp_text value "BNO055" (at 0 19.05 -90 unlocked) (layer "F.Fab")
         (effects (font (size 1 1) (thickness 0.15)))
     )
@@
         (effects (font (size 1 1) (thickness 0.15)))
     )
-    (fp_text value "0.1μF" (at 0 1.43 90) (layer "F.Fab")
+    (fp_text value "0.1uF" (at 0 1.43 90) (layer "F.Fab")
         (effects (font (size 1 1) (thickness 0.15)))
     )
@@
         (effects (font (size 1 1) (thickness 0.153)))
     )
-    (fp_text value "4.7kΩ" (at 0 1.43 90) (layer "F.Fab")
+    (fp_text value "4.7kR" (at 0 1.43 90) (layer "F.Fab")
         (effects (font (size 1 1) (thickness 0.15)))
     )
@@
         (effects (font (size 1 1) (thickness 0.15)))
     )
-    (fp_text value "10kΩ" (at 0 1.65 90) (layer "F.Fab")
+    (fp_text value "10kR" (at 0 1.65 90) (layer "F.Fab")
         (effects (font (size 1 1) (thickness 0.15)))
     )
@@
         (effects (font (size 1 1) (thickness 0.15)))
     )
-    (fp_text value "47μF" (at 0 4.35 90) (layer "F.Fab")
+    (fp_text value "47uF" (at 0 4.35 90) (layer "F.Fab")
         (effects (font (size 1 1) (thickness 0.15)))
     )
@@
         (effects (font (size 1 1) (thickness 0.153)))
     )
-    (fp_text value "120Ω" (at 0 1.43 -90) (layer "F.Fab")
+    (fp_text value "120R" (at 0 1.43 -90) (layer "F.Fab")
         (effects (font (size 1 1) (thickness 0.15)))
     )
@@
         (effects (font (size 1 1) (thickness 0.153)))
     )
-    (fp_text value "300Ω" (at 0 1.43 90) (layer "F.Fab")
-        (effects (font (size 1 1) (thickness 0.15)))
-    )
+    (fp_text value "300R" (at 0 1.43 90) (layer "F.Fab")
+        (effects (font (size 1 1) (thickness 0.15)))
+    )

Commit message: QRと署名を更新
Parts:
- removed the G*** at (148.0, 60.5)
- added G***: LOGO, LOGO, F.Cu at (145.5, 137.0)
- added G***: LOGO, LOGO, B.Cu at (148.5, 60.0)
Routing:
- net GND: vias 169 -> 168
Other:
- board text added: "Sensing Module Build 2"
- board text removed: "Sensing Module Build 1"

Commit message: ガーバーを再出力
Parts:
- removed the G*** at (145.5, 137.0)
