File: Projects/KiCad/THRControlModule/MAX31856.kicad_sch (KiCad schematic)
At the start: 17 parts, among them J3 Screw_Terminal_01x02, U4 MAX31856MUD+T

Commit message: 基板を更新
Parts:
- C10: renamed from C8; value C -> 0.01u; footprint (none) -> Capacitor_SMD:C_0603_1608Metric_Pad1.08x0.95mm_HandSolder
- C11: renamed from C7; value C -> 0.1u; footprint (none) -> Capacitor_SMD:C_0603_1608Metric_Pad1.08x0.95mm_HandSolder
- C12: renamed from C9; value C -> 0.01u; footprint (none) -> Capacitor_SMD:C_0603_1608Metric_Pad1.08x0.95mm_HandSolder
- C13: renamed from C10; value C -> 0.1u; footprint (none) -> Capacitor_SMD:C_0603_1608Metric_Pad1.08x0.95mm_HandSolder
- C14: renamed from C11; value C -> 0.1u; footprint (none) -> Capacitor_SMD:C_0603_1608Metric_Pad1.08x0.95mm_HandSolder
- D1, D2, D3: footprint (none) -> Diode_SMD:D_SOD-123
- J6: renamed from J3; footprint (none) -> MAX31856MUD_T:RS_PRO_611-8157
- R11: renamed from R5; value R -> 100; footprint (none) -> Resistor_SMD:R_0805_2012Metric_Pad1.20x1.40mm_HandSolder
- R12: renamed from R6; value R -> 100; footprint (none) -> Resistor_SMD:R_0805_2012Metric_Pad1.20x1.40mm_HandSolder
- R13: renamed from R7; value R -> 10k; footprint (none) -> Resistor_SMD:R_0603_1608Metric_Pad0.98x0.95mm_HandSolder
- R14: renamed from R8; value R -> 10k; footprint (none) -> Resistor_SMD:R_0603_1608Metric_Pad0.98x0.95mm_HandSolder
- R15: renamed from R9; value R -> 10k; footprint (none) -> Resistor_SMD:R_0603_1608Metric_Pad0.98x0.95mm_HandSolder
- renumbered U4 to U3

Commit message: 基板を更新（最終確認中）
Parts:
- renumbered C13 to C11, C14 to C12, C10 to C13, C11 to C14, C12 to C15, D1 to D6, D2 to D7, D3 to D8, R15 to R17, R11 to R18, R14 to R19, R13 to R20, R12 to R21
