File: Projects/KiCad/THRControlModule/THRControlModule.kicad_sch (KiCad schematic)
At the start: 7 parts, among them IC1 LTC1480CN8#PBF, IC2 LTC1480CN8#PBF

Commit message: Kicadプラグインのgifを追加
Parts:
- removed D1: D, symbol Device:D
Connections:
- net +12V: now also A1.30 (VIN)
- net +3.3V: now also A1.17 (3V3)
- net +5V: now reaches A1.27 (+5V)
Changed lines of the file:
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@@
+    (stroke (width 0) (type default))
+  )
+  (wire (pts (xy 143.51 71.12) (xy 143.51 74.93))
     (stroke (width 0) (type default))
   )
@@
     (stroke (width 0) (type default))
   )
-  (wire (pts (xy 135.89 72.39) (xy 135.89 74.93))
-    (stroke (width 0) (type default))
-  )
   (wire (pts (xy 71.12 109.22) (xy 71.12 106.68))
     (stroke (width 0) (type default))
@@
     (stroke (width 0) (type default))
   )
-  (wire (pts (xy 135.89 63.5) (xy 135.89 64.77))
+  (wire (pts (xy 135.89 63.5) (xy 135.89 74.93))
     (stroke (width 0) (type default))
   )
@@
   )
   (wire (pts (xy 68.58 96.52) (xy 69.85 96.52))
+    (stroke (width 0) (type default))
+  )
+  (wire (pts (xy 140.97 66.04) (xy 140.97 74.93))
     (stroke (width 0) (type default))
   )
@@
     )
   )
-  (symbol (lib_id "Device:D") (at 135.89 68.58 90) (unit 1)
-    (in_bom yes) (on_board yes) (dnp no) (fields_autoplaced)
-    (property "Reference" "D1" (at 138.43 67.945 90)
-      (effects (font (size 1.27 1.27)) (justify right))
-    )
-    (property "Value" "D" (at 138.43 70.485 90)
-      (effects (font (size 1.27 1.27)) (justify right))
-    )
-    (property "Footprint" "" (at 135.89 68.58 0)
-      (effects (font (size 1.27 1.27)) hide)
-    )
-    (property "Datasheet" "~" (at 135.89 68.58 0)
-      (effects (font (size 1.27 1.27)) hide)
-    )
-    (property "Sim.Device" "D" (at 135.89 68.58 0)
-      (effects (font (size 1.27 1.27)) hide)
-    )
-    (property "Sim.Pins" "1=K 2=A" (at 135.89 68.58 0)
+  (symbol (lib_id "power:+3.3V") (at 67.31 25.4 0) (unit 1)
+    (in_bom yes) (on_board yes) (dnp no) (fields_autoplaced)
+    (property "Reference" "#PWR02" (at 67.31 29.21 0)
+      (effects (font (size 1.27 1.27)) hide)
+    )
+    (property "Value" "+3.3V" (at 67.31 21.59 0)
+      (effects (font (size 1.27 1.27)))
+    )
+    (property "Footprint" "" (at 67.31 25.4 0)
+      (effects (font (size 1.27 1.27)) hide)
+    )
+    (property "Datasheet" "" (at 67.31 25.4 0)
+      (effects (font (size 1.27 1.27)) hide)
+    )
+    (pin "1")
+    (instances
+      (project "THRControlModule"
+        (path "/93cdfa36-4bed-45c7-a4a4-3a03363a12aa"
+          (reference "#PWR02") (unit 1)
+        )
+      )
+    )
+  )
+  (symbol (lib_id "Device:C") (at 72.39 30.48 90) (unit 1)
+    (in_bom yes) (on_board yes) (dnp no) (fields_autoplaced)
+    (property "Reference" "C1" (at 72.39 24.13 90)
+      (effects (font (size 1.27 1.27)))
+    )
+    (property "Value" "C" (at 72.39 26.67 90)
+      (effects (font (size 1.27 1.27)))
+    )
+    (property "Footprint" "" (at 76.2 29.5148 0)
+      (effects (font (size 1.27 1.27)) hide)
+    )
+    (property "Datasheet" "~" (at 72.39 30.48 0)
       (effects (font (size 1.27 1.27)) hide)
     )
@@
       (project "THRControlModule"
         (path "/93cdfa36-4bed-45c7-a4a4-3a03363a12aa"
-          (reference "D1") (unit 1)
-        )
-      )
-    )
-  )
-  (symbol (lib_id "power:+3.3V") (at 67.31 25.4 0) (unit 1)
-    (in_bom yes) (on_board yes) (dnp no) (fields_autoplaced)
-    (property "Reference" "#PWR02" (at 67.31 29.21 0)
-      (effects (font (size 1.27 1.27)) hide)
-    )
-    (property "Value" "+3.3V" (at 67.31 21.59 0)
-      (effects (font (size 1.27 1.27)))
-    )
-    (property "Footprint" "" (at 67.31 25.4 0)
-      (effects (font (size 1.27 1.27)) hide)
-    )
-    (property "Datasheet" "" (at 67.31 25.4 0)
-      (effects (font (size 1.27 1.27)) hide)
-    )
-    (pin "1")
-    (instances
-      (project "THRControlModule"
-        (path "/93cdfa36-4bed-45c7-a4a4-3a03363a12aa"
-          (reference "#PWR02") (unit 1)
-        )
-      )
-    )
-  )
-  (symbol (lib_id "Device:C") (at 72.39 30.48 90) (unit 1)
-    (in_bom yes) (on_board yes) (dnp no) (fields_autoplaced)
-    (property "Reference" "C1" (at 72.39 24.13 90)
-      (effects (font (size 1.27 1.27)))
-    )
-    (property "Value" "C" (at 72.39 26.67 90)
-      (effects (font (size 1.27 1.27)))
-    )
-    (property "Footprint" "" (at 76.2 29.5148 0)
-      (effects (font (size 1.27 1.27)) hide)
-    )
-    (property "Datasheet" "~" (at 72.39 30.48 0)
-      (effects (font (size 1.27 1.27)) hide)
-    )
-    (pin "1")
-    (pin "2")
-    (instances
-      (project "THRControlModule"
-        (path "/93cdfa36-4bed-45c7-a4a4-3a03363a12aa"
           (reference "C1") (unit 1)
         )
       )
+    )
+  )
+  (symbol (lib_id "power:+5V") (at 143.51 71.12 0) (unit 1)
+    (in_bom yes) (on_board yes) (dnp no) (fields_autoplaced)
+    (property "Reference" "#PWR09" (at 143.51 74.93 0)
+      (effects (font (size 1.27 1.27)) hide)
+    )
+    (property "Value" "+5V" (at 143.51 67.31 0)
+      (effects (font (size 1.27 1.27)))
+    )
+    (property "Footprint" "" (at 143.51 71.12 0)
+      (effects (font (size 1.27 1.27)) hide)
+    )
+    (property "Datasheet" "" (at 143.51 71.12 0)
+      (effects (font (size 1.27 1.27)) hide)
+    )
+    (pin "1")
+    (instances
+      (project "THRControlModule"
+        (path "/93cdfa36-4bed-45c7-a4a4-3a03363a12aa"
+          (reference "#PWR09") (unit 1)
+        )
+      )
+    )
+  )
+  (symbol (lib_id "power:+3.3V") (at 140.97 66.04 0) (unit 1)
+    (in_bom yes) (on_board yes) (dnp no) (fields_autoplaced)
+    (property "Reference" "#PWR08" (at 140.97 69.85 0)
+      (effects (font (size 1.27 1.27)) hide)
+    )
+    (property "Value" "+3.3V" (at 140.97 62.23 0)
+      (effects (font (size 1.27 1.27)))
+    )
+    (property "Footprint" "" (at 140.97 66.04 0)
+      (effects (font (size 1.27 1.27)) hide)
+    )
+    (property "Datasheet" "" (at 140.97 66.04 0)
+      (effects (font (size 1.27 1.27)) hide)
+    )
+    (pin "1")
+    (instances
+      (project "THRControlModule"
+        (path "/93cdfa36-4bed-45c7-a4a4-3a03363a12aa"
+          (reference "#PWR08") (unit 1)
+        )
+      )

Commit message: 基板を更新
Parts:
- added C12, C13, C14: 0.1u, symbol Device:C
- added C3, C4, C5, C6: C, symbol Device:C
- added J1, J2, J4: Conn_01x04, symbol Connector_Generic:Conn_01x04
- added J5: Conn_01x06, symbol Connector_Generic:Conn_01x06
- added J6: Conn_01x08, symbol Connector_Generic:Conn_01x08
- added LS1: PKB24SPCH3601-B0, PKB24SPCH3601-B0:SPKR_PKB24SPCH3601-B0, symbol PKB24SPCH3601-B0:PKB24SPCH3601-B0
- added R10, R12, R14: 10k, symbol Device:R
- added R11, R13, R15: 1k, symbol Device:R
- added R2, R3, R4: R, symbol Device:R
- added U1: MCP2515-I/P, MCP2515-I_P:DIP254P762X432-18, symbol MCP2515-I_P:MCP2515-I/P
- added U2: MCP2562-E-P, Package_DIP:DIP-8_W7.62mm, symbol Interface_CAN_LIN:MCP2562-E-P
- added Y1: Crystal, symbol Device:Crystal
- IC1, IC2: footprint DIP794W53P254L1016H394Q8N -> LTC1480CN8#PBF:DIP794W53P254L1016H394Q8N
- R1: value R -> 120
Connections:
- net +12V: now also J1.2 (Pin_2), J2.2 (Pin_2), J6.1 (Pin_1), J6.2 (Pin_2)
- net +5V: now also C6.1, J5.6 (Pin_6), U2.3 (VDD), U2.5 (Vio)
- net GND: now also A1.29 (GND), A1.4 (GND), C12.2, C13.2, C14.2, C3.1, C4.2, C5.2, C6.2, J1.1 (Pin_1), J2.1 (Pin_1), J4.1 (Pin_1), J4.3 (Pin_3), J5.4 (Pin_4), J6.3 (Pin_3), J6.4 (Pin_4), LS1.N, U1.9 (VSS), U2.2 (VSS), U2.8 (STBY)
- net RS485__A1: now also IC1.6 (A), J1.3 (Pin_3), R2.2
- net RS485__A2: now also J2.3 (Pin_3)
- net RS485__B1: now also IC1.7 (B), J1.4 (Pin_4), R2.1
- net RS485__B2: now also J2.4 (Pin_4)
- net Umbilical__LaunchPin: now reaches A1.10 (D7)
- net Umbilical__LaunchPin: now also R13.2
- net Umbilical__WaitingPin: now reaches A1.11 (D8)
- net Umbilical__WaitingPin: now also R11.2
- net MAX31856__DRDY-DRDY: now reaches A1.12 (D9)
- net MAX31856__FAULT-FAULT: now reaches A1.13 (D10)
- net SPI__MOSI: now reaches A1.14 (MOSI)
- net SPI__MOSI: now also U1.14 (SI)
- net SPI__MISO: now reaches A1.15 (MISO)
- net SPI__MISO: now also J5.3 (Pin_3), U1.15 (SO)
- net SPI__SCLK: now reaches A1.16 (SCK)
- net SPI__SCLK: now also J5.1 (Pin_1), U1.13 (SCK)
- net B3M_Servo__Open: now reaches A1.19 (A0)
- net B3M_Servo__Open: now also R15.2
- net B3M_Servo__Close: now reaches A1.20 (A1)
- net RS405_Servo__Open: now reaches A1.21 (A2)
- net RS405_Servo__Close: now reaches A1.22 (A3)
- net IO__Busser: now reaches A1.25 (A6)
- net IO__Busser: now also LS1.P
- net MAX31856__~{CS}-~{CS}: now reaches A1.7 (D4)
- net MAX31855__~{CS}-~{CS}: now reaches A1.8 (D5)
- net MAX31855__~{CS}-~{CS}: now also J5.2 (Pin_2)
- net MCP2515__~{CS}-~{CS}: now reaches A1.9 (D6)
- net MCP2515__~{CS}-~{CS}: now also U1.16 (~CS)
- new net: C14.1, R14.2, R15.1
- new net: C13.1, R12.2, R13.1
- new net: R3.2, U1.17 (~RESET)
- new net: C12.1, R10.2, R11.1
- new net +3V3: C3.2, R3.1, U1.18 (VDD)
- new net B3M_Servo__OpenInput: R14.1
- new net CAN__H: J6.7 (Pin_7), J6.8 (Pin_8), R4.1, U2.7 (CANH)
- new net CAN__L: J6.5 (Pin_5), J6.6 (Pin_6), R4.2, U2.6 (CANL)
- new net CAN__RXD-CANRX: U1.2 (RXCAN), U2.4 (RXD)
- new net CAN__TXD-TXCAN: U1.1 (TXCAN), U2.1 (TXD)
- new net OCS1: C4.1, U1.8 (OSC1), Y1.1
- new net OCS2: C5.1, U1.7 (OSC2), Y1.2
- new net Umbilical__LaunchPinInput: J4.4 (Pin_4), R12.1
- new net Umbilical__WaitingPinInput: J4.2 (Pin_2), R10.1
- no-connect marks 0 -> 14
Other:
- added sheet MAX31856 (MAX31856.kicad_sch)
- moved on the sheet: A1, C2, IC2, R1

Commit message: 基板を更新
Parts:
- added H1, H2, H3, H4: MountingHole, MountingHole:MountingHole_4.5mm, symbol Mechanical:MountingHole
- C1: renamed from C12; footprint (none) -> Capacitor_SMD:C_0603_1608Metric_Pad1.08x0.95mm_HandSolder
- C2: renamed from C13; footprint (none) -> Capacitor_SMD:C_0603_1608Metric_Pad1.08x0.95mm_HandSolder
- C3: renamed from C14; footprint (none) -> Capacitor_SMD:C_0603_1608Metric_Pad1.08x0.95mm_HandSolder
- C4: renamed from C1; value C -> 0.1u; footprint (none) -> Capacitor_SMD:C_0603_1608Metric_Pad1.08x0.95mm_HandSolder
- C5: renamed from C2; value C -> 0.1u; footprint (none) -> Capacitor_SMD:C_0603_1608Metric_Pad1.08x0.95mm_HandSolder
- C6: value C -> 0.1u; footprint (none) -> Capacitor_SMD:C_0603_1608Metric_Pad1.08x0.95mm_HandSolder
- C7: renamed from C3; value C -> 0.1u; footprint (none) -> Capacitor_SMD:C_0603_1608Metric_Pad1.08x0.95mm_HandSolder
- C8: renamed from C4; value C -> 15p; footprint (none) -> Capacitor_SMD:C_0603_1608Metric_Pad1.08x0.95mm_HandSolder
- C9: renamed from C5; value C -> 15p; footprint (none) -> Capacitor_SMD:C_0603_1608Metric_Pad1.08x0.95mm_HandSolder
- J4: renamed from J6; footprint (none) -> Hirose_Connector:Hirose_DF11B-8DP-2DS
- R1: renamed from R10; footprint (none) -> Resistor_SMD:R_0603_1608Metric_Pad0.98x0.95mm_HandSolder
- R10: renamed from R3; value R -> 10k; footprint (none) -> Resistor_SMD:R_0603_1608Metric_Pad0.98x0.95mm_HandSolder
- R2: renamed from R12; footprint (none) -> Resistor_SMD:R_0603_1608Metric_Pad0.98x0.95mm_HandSolder
- R3: renamed from R14; footprint (none) -> Resistor_SMD:R_0603_1608Metric_Pad0.98x0.95mm_HandSolder
- R4: renamed from R11; footprint (none) -> Resistor_SMD:R_0603_1608Metric_Pad0.98x0.95mm_HandSolder
- R5: renamed from R13; footprint (none) -> Resistor_SMD:R_0603_1608Metric_Pad0.98x0.95mm_HandSolder
- R6: renamed from R15; footprint (none) -> Resistor_SMD:R_0603_1608Metric_Pad0.98x0.95mm_HandSolder
- R7: renamed from R2; value R -> 120; footprint (none) -> Resistor_SMD:R_0603_1608Metric_Pad0.98x0.95mm_HandSolder
- R8: renamed from R1; footprint (none) -> Resistor_SMD:R_0603_1608Metric_Pad0.98x0.95mm_HandSolder
- R9: renamed from R4; value R -> 120; footprint (none) -> Resistor_SMD:R_0603_1608Metric_Pad0.98x0.95mm_HandSolder
- Y1: value Crystal -> 8MHz; footprint (none) -> Crystal:Crystal_HC49-U_Vertical
- renumbered J4 to J3, U2 to U1, U1 to U2
Connections:
- net +3.3V: now also C7.2, U2.18 (VDD)
- net +3V3: no longer C7.2, U2.18 (VDD)
Other:
- moved on the sheet: LS1

Commit message: DF1Bシリーズとしてまとめた。
Parts:
- added D1: D, Diode_SMD:D_SOD-123, symbol Device:D
- added D5: LED, LED_SMD:LED_0603_1608Metric_Pad1.05x0.95mm_HandSolder, symbol Device:LED
- added R16: 1k, Resistor_SMD:R_0603_1608Metric_Pad0.98x0.95mm_HandSolder, symbol Device:R
- J1, J2, J3: footprint (none) -> Hirose_Connector:Hirose_DF1BZ-4P-2.5DS
- J5: footprint (none) -> Hirose_Connector:DF1BZ-6P-2.5DS
- Y1: footprint Crystal:Crystal_HC49-U_Vertical -> Crystal:Crystal_HC49-4H_Vertical
Connections:
- net +3V3 is gone; now on net +3.3V: R10.1
- net +12V: now also D1.1 (K), D1.2 (A), R16.1
- net GND: now also D5.1 (K)
- new net: D5.2 (A), R16.2

Commit message: Kicadの更新
Parts:
- removed J5: Conn_01x06, Hirose_Connector:DF1BZ-6P-2.5DS, symbol Connector_Generic:Conn_01x06
- added C15: 0.1u, Capacitor_SMD:C_0603_1608Metric_Pad1.08x0.95mm_HandSolder, symbol Device:C
- added J5: Conn_01x04, Hirose_Connector:Hirose_DF1BZ-4P-2.5DS, symbol Connector_Generic:Conn_01x04
- added R17: 10k, Resistor_SMD:R_0603_1608Metric_Pad0.98x0.95mm_HandSolder, symbol Device:R
- added R18: 1k, Resistor_SMD:R_0603_1608Metric_Pad0.98x0.95mm_HandSolder, symbol Device:R
Connections:
- net B3M_Servo__Close: now also R18.2
- net B3M_Servo__OpenInput: now also J5.2 (Pin_2)
- net GND: now also J5.1 (Pin_1)
- net MAX31855__~{CS}-~{CS}: no longer names the net of A1.8 (D5)
- net RS405_Servo__Close: no longer names the net of A1.22 (A3)
- net RS405_Servo__Open: no longer names the net of A1.21 (A2)
- new net: C15.1, R17.2, R18.1
- new net B3M_Servo__CloseInput: J5.3 (Pin_3), R17.1
- no-connect marks 14 -> 16
Other:
- moved on the sheet: C1, C2, C3, C4, C5, C6, D1, D5, IC1, IC2, J1, J2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

Commit message: 基板を更新（最終確認中）
Parts:
- added D1, D2, D3: LED, LED_SMD:LED_0603_1608Metric_Pad1.05x0.95mm_HandSolder, symbol Device:LED
- added R1, R2, R4: 1k, Resistor_SMD:R_0603_1608Metric_Pad0.98x0.95mm_HandSolder, symbol Device:R
- renumbered C4 to C1, C15 to C10, C5 to C2, C7 to C3, C1 to C4, C8 to C5, C9 to C6, C2 to C7, C6 to C8, C3 to C9, R2 to R10, R5 to R11, R3 to R12, R6 to R13, R9 to R14, R17 to R15, R18 to R16, R7 to R3, R8 to R5, R1 to R6, R4 to R7, R10 to R8, R16 to R9, U2 to U1, U1 to U2
Connections:
- net +12V: no longer A1.30 (VIN), D1.1 (K)
- net B3M_Servo__CloseInput: now also J5.4 (Pin_4); no longer J5.3 (Pin_3)
- net GND: now also C10.2, J5.3 (Pin_3), D1.1 (K), D2.1 (K), D3.1 (K)
- net O__OrangeLED: now reaches A1.21 (A2)
- net O__OrangeLED: now also R1.1
- net O__RedLED: now reaches A1.22 (A3)
- net O__RedLED: now also R2.1
- net O__BlueLED: now reaches A1.26 (A7)
- net O__BlueLED: now also R4.1
- new net: D1.2 (A), R1.2
- new net: D3.2 (A), R4.2
- new net: D2.2 (A), R2.2
- new net 12Vin: A1.30 (VIN), D1.1 (K)
- no-connect marks 16 -> 13
Other:
- moved on the sheet: C1, D1, D5, R9
